File: KiCadProjects/Fonte_Tensao/Fonte_tensao_LM675_v04/Fonte_tensao_LM675_v04.kicad_pcb (KiCad board)
At the start: 2 copper layers, 90 x 100 mm, 30 parts, among them J1 Barrel_Jack, J2 sinais analogicos, J3 comunicacao / sinais digitais, J4 tensoes, U1 L7809, U2 LM7909_TO220, U3 LM675, U4 L7805, U5 L7905, U6 LM1117T-3.3

Commit message: revisao de  v03 para os componentes utilizados no primeiro  prototipo
Parts:
- added C3: 0.1uf, Capacitor_THT:CP_Radial_D5.0mm_P2.50mm, F.Cu at (126.1, 135.8)
- added C6: 0.1uF, Capacitor_THT:CP_Radial_D5.0mm_P2.50mm, F.Cu at (136.8, 120.6)
- C1: value 0.33uF -> 3.3uF
- C10, C11: value 10uF -> 100uF
- C2: value 2.2uF -> 22uF
- C4, C8: value 0.1uF -> 1uF
- R1: value 1k -> 470
Connections:
- D5 pad 1: GND -> Earth
Routing:
- net Net-(U3-V-): track 0.00 -> 41.8 mm
- net GND: track 403.1 -> 375.4 mm
- net switch: track 234.9 -> 238.1 mm

Commit message: Fonte de tensao v04 - Para fabricacao do segundo prototipo
Parts:
- removed C3: 0.1uf, Capacitor_THT:CP_Radial_D5.0mm_P2.50mm
- removed C6: 0.1uF, Capacitor_THT:CP_Radial_D5.0mm_P2.50mm
- removed U3: LM675, Package_TO_SOT_THT:TO-220-5_P3.4x3.7mm_StaggerOdd_Lead3.8mm_Vertical
- R1, R2, R3, R4, R5, R6: footprint Resistor_THT:R_Axial_DIN0617_L17.0mm_D6.0mm_P20.32mm_Horizontal -> Resistor_THT:R_Axial_DIN0207_L6.3mm_D2.5mm_P7.62mm_Horizontal
Connections:
- net GND renamed VEE
Routing:
- net switch: track 238.1 -> 104.4 mm, vias 9 -> 8
- net VEE: track 375.4 -> 264.7 mm
- net +3.3V: track 145.3 -> 36.0 mm
- net Earth: track 321.9 -> 233.2 mm
- net Net-(U3-+): track 47.2 -> 0.36 mm
- net Net-(C7-Pad1): track 46.5 -> 0.00 mm
- net Net-(U3-V-): track 41.8 -> 0.00 mm
- net Net-(U3--): track 39.1 -> 0.00 mm
- net Net-(D5-A): track 35.2 -> 0.00 mm
