File: KiCadProjects/Fonte_Corrente_Monopolar/Fonte_corrente_mono.kicad_pcb (KiCad board)
At the start: 2 copper layers, 90 x 100 mm, 24 parts, among them J1 Vref, J2 tensoes, J3 sinais analogicos, J4 comunicacao / sinais digitais, J5 Vref, U1-howland1 AD828AN, U2 INA128, U3-cond1 AD828AN

Commit message: alterações PCB
Parts:
- removed J5: Vref, Connector_PinHeader_2.54mm:PinHeader_1x03_P2.54mm_Vertical
Connections:
- J1 pad 2: Net-(J1-Pin_2) -> Net-(D1-K)
- R10 pad 1: Net-(J1-Pin_2) -> Net-(D1-K)
Routing:
- net Net-(D1-K): track 20.0 -> 63.0 mm
- net Net-(J1-Pin_2): track 35.5 -> 0.00 mm
- net +3.3V: track 174.4 -> 162.9 mm
- net +5V: track 131.2 -> 123.7 mm
- net out_corrente: track 104.7 -> 102.9 mm
- net Net-(U1-howland1--IN2): track 24.1 -> 22.5 mm
- net Earth: track 243.1 -> 244.0 mm
- net +9V: track 152.0 -> 151.1 mm
