File: KiCadProjects/Condicionamento/condicionamento_BIA_v01/condicionamento_BIA_v01.kicad_pcb (KiCad board)
At the start: 2 copper layers, 90 x 100 mm, 3 parts, among them J2 tensoes, J3 sinais analogicos, J4 comunicacao / sinais digitais

Commit message: condicionamento
Parts:
- added Brd1: SSD1306, SSD1306:128x64OLED, F.Cu at (147.3, 127.0)
- added C1: 1 uF, Capacitor_THT:CP_Radial_D5.0mm_P2.50mm, F.Cu at (139.7, 59.7)
- added C2: 470 pF, Capacitor_THT:CP_Radial_D5.0mm_P2.50mm, F.Cu at (142.2, 87.6)
- added C3: 1 uF, Capacitor_THT:CP_Radial_D5.0mm_P2.50mm, F.Cu at (162.6, 59.7)
- added C4: 470 pF, Capacitor_THT:CP_Radial_D5.0mm_P2.50mm, F.Cu at (157.5, 87.6)
- added D1: 1N5819, Diode_THT:D_DO-41_SOD81_P10.16mm_Horizontal, F.Cu at (124.5, 67.3)
- added D2: 1N5819, Diode_THT:D_DO-41_SOD81_P10.16mm_Horizontal, F.Cu at (132.1, 92.7)
- added D3: 1N5819, Diode_THT:D_DO-41_SOD81_P10.16mm_Horizontal, F.Cu at (177.8, 67.3)
- added D4: 1N5819, Diode_THT:D_DO-41_SOD81_P10.16mm_Horizontal, F.Cu at (170.2, 92.7)
- added J1: Vref, Connector_PinHeader_2.54mm:PinHeader_1x03_P2.54mm_Vertical, F.Cu at (116.8, 53.3)
- added J5: sinais_condicionados, Connector_PinHeader_2.54mm:PinHeader_1x04_P2.54mm_Horizontal, F.Cu at (151.1, 148.0)
- added R1: 100k, Resistor_THT:R_Axial_DIN0207_L6.3mm_D2.5mm_P7.62mm_Horizontal, F.Cu at (130.8, 59.7)
- added R2: 100k, Resistor_THT:R_Axial_DIN0207_L6.3mm_D2.5mm_P7.62mm_Horizontal, F.Cu at (137.2, 72.4)
- added R3: 220, Resistor_THT:R_Axial_DIN0207_L6.3mm_D2.5mm_P7.62mm_Horizontal, F.Cu at (137.2, 77.5)
- added R4: 100k, Resistor_THT:R_Axial_DIN0207_L6.3mm_D2.5mm_P7.62mm_Horizontal, F.Cu at (171.4, 59.7)
- added R5: 100k, Resistor_THT:R_Axial_DIN0207_L6.3mm_D2.5mm_P7.62mm_Horizontal, F.Cu at (163.8, 72.4)
- added R6: 220, Resistor_THT:R_Axial_DIN0207_L6.3mm_D2.5mm_P7.62mm_Horizontal, F.Cu at (163.8, 77.5)
- added R7: 4k7, Resistor_THT:R_Axial_DIN0207_L6.3mm_D2.5mm_P7.62mm_Horizontal, F.Cu at (153.7, 96.5)
- added R8: 4k7, Resistor_THT:R_Axial_DIN0207_L6.3mm_D2.5mm_P7.62mm_Horizontal, F.Cu at (153.7, 104.1)
- added U1: AD828AN, footprints:N_8_ADI, F.Cu at (146.8, 54.7)
- added U2: BluePill_STM32F103C, BluePill_breakouts:BluePill_STM32F103C, F.Cu at (114.3, 99.1)
- added U3: BluePill_STM32F103C, BluePill_breakouts:BluePill_STM32F103C, F.Cu at (165.1, 99.1)
Connections:
- net +12V renamed VCC
- net -12V renamed VEE
- net Ampl2 renamed AmpI2
- J3 pad 22: Ampl1 -> AmpI1
- J4 pad 22: X9x10x_INC -> unconnected-(J4-Pin_22-Pad22)
- J4 pad 23: X9x10x_U/D -> unconnected-(J4-Pin_23-Pad23)
Routing:
- net Earth: track 0.00 -> 182.4 mm
- net Amp_E2: track 0.00 -> 45.4 mm
- net Net-(D1-A): track 0.00 -> 43.4 mm
- net nó4: track 0.00 -> 25.8 mm
- net nó2: track 0.00 -> 24.5 mm
- net Vref: track 0.00 -> 21.2 mm
- net nó3: track 0.00 -> 10.7 mm
- net nó1: track 0.00 -> 8.20 mm

Commit message: PCB
Parts:
- removed Brd1: SSD1306, SSD1306:128x64OLED
- removed C1, C3: 1 uF, Capacitor_THT:CP_Radial_D5.0mm_P2.50mm
- removed C2, C4: 470 pF, Capacitor_THT:CP_Radial_D5.0mm_P2.50mm
- removed D1, D2, D3, D4: 1N5819, Diode_THT:D_DO-41_SOD81_P10.16mm_Horizontal
- removed J1: Vref, Connector_PinHeader_2.54mm:PinHeader_1x03_P2.54mm_Vertical
- removed J5: sinais_condicionados, Connector_PinHeader_2.54mm:PinHeader_1x04_P2.54mm_Horizontal
- removed R1, R2, R4, R5: 100k, Resistor_THT:R_Axial_DIN0207_L6.3mm_D2.5mm_P7.62mm_Horizontal
- removed R3, R6: 220, Resistor_THT:R_Axial_DIN0207_L6.3mm_D2.5mm_P7.62mm_Horizontal
- removed R7, R8: 4k7, Resistor_THT:R_Axial_DIN0207_L6.3mm_D2.5mm_P7.62mm_Horizontal
- removed U1: AD828AN, footprints:N_8_ADI
- removed U2, U3: BluePill_STM32F103C, BluePill_breakouts:BluePill_STM32F103C
Routing:
- net Earth: track 182.4 -> 0.00 mm
- net Amp_E2: track 45.4 -> 0.00 mm
- net Net-(D1-A): track 43.4 -> 0.00 mm
- net nó4: track 25.8 -> 0.00 mm
- net nó2: track 24.5 -> 0.00 mm
- net Vref: track 21.2 -> 0.00 mm
- net nó3: track 10.7 -> 0.00 mm
- net nó1: track 8.20 -> 0.00 mm

Commit message: PCB
Parts:
- added Brd1: SSD1306, SSD1306:128x64OLED, F.Cu at (145.0, 157.5)
- added C1: 1 uF, Capacitor_THT:CP_Radial_D5.0mm_P2.50mm, F.Cu at (115.2, 62.0)
- added C2: 470 pF, Capacitor_THT:CP_Radial_D5.0mm_P2.50mm, F.Cu at (178.8, 73.7)
- added C3: 1 uF, Capacitor_THT:CP_Radial_D5.0mm_P2.50mm, F.Cu at (129.3, 62.0)
- added C4: 470 pF, Capacitor_THT:CP_Radial_D5.0mm_P2.50mm, F.Cu at (171.6, 61.6)
- added D1: 1N5819, Diode_THT:D_DO-41_SOD81_P10.16mm_Horizontal, F.Cu at (149.2, 82.8)
- added D2: 1N5819, Diode_THT:D_DO-41_SOD81_P10.16mm_Horizontal, F.Cu at (140.1, 89.2)
- added D3: 1N5819, Diode_THT:D_DO-41_SOD81_P10.16mm_Horizontal, F.Cu at (156.5, 89.7)
- added D4: 1N5819, Diode_THT:D_DO-41_SOD81_P10.16mm_Horizontal, F.Cu at (156.7, 71.2)
- added J1: Vref, Connector_PinHeader_2.54mm:PinHeader_1x03_P2.54mm_Vertical, F.Cu at (121.9, 82.2)
- added J5: sinais_condicionados, Connector_PinHeader_2.54mm:PinHeader_1x04_P2.54mm_Horizontal, F.Cu at (145.0, 54.0)
- added J6: alimetacao_Master, Connector_PinHeader_2.54mm:PinHeader_1x02_P2.54mm_Vertical, F.Cu at (166.5, 52.8)
- added J7: Eletrodos, Connector_PinHeader_2.54mm:PinHeader_1x02_P2.54mm_Horizontal, F.Cu at (132.0, 54.1)
- added R1: 100k, Resistor_THT:R_Axial_DIN0207_L6.3mm_D2.5mm_P7.62mm_Horizontal, F.Cu at (118.4, 84.2)
- added R2: 100k, Resistor_THT:R_Axial_DIN0207_L6.3mm_D2.5mm_P7.62mm_Horizontal, F.Cu at (115.4, 67.6)
- added R3: 220, Resistor_THT:R_Axial_DIN0207_L6.3mm_D2.5mm_P7.62mm_Horizontal, F.Cu at (132.2, 93.8)
- added R4: 100k, Resistor_THT:R_Axial_DIN0207_L6.3mm_D2.5mm_P7.62mm_Horizontal, F.Cu at (143.8, 82.0)
- added R5: 100k, Resistor_THT:R_Axial_DIN0207_L6.3mm_D2.5mm_P7.62mm_Horizontal, F.Cu at (135.2, 86.2)
- added R6: 220, Resistor_THT:R_Axial_DIN0207_L6.3mm_D2.5mm_P7.62mm_Horizontal, F.Cu at (132.2, 66.8)
- added R7: 4k7, Resistor_THT:R_Axial_DIN0207_L6.3mm_D2.5mm_P7.62mm_Horizontal, F.Cu at (140.2, 115.4)
- added R8: 4k7, Resistor_THT:R_Axial_DIN0207_L6.3mm_D2.5mm_P7.62mm_Horizontal, F.Cu at (148.0, 131.8)
- added U1: AD828AN, AD828:N_8_ADI, F.Cu at (118.7, 62.5)
- added U2: BluePill_STM32F103C, BluePill_breakouts:BluePill_STM32F103C, F.Cu at (164.8, 98.4)
- added U3: BluePill_STM32F103C, BluePill_breakouts:BluePill_STM32F103C, F.Cu at (112.3, 99.4)
Routing:
- net Earth: track 0.00 -> 214.3 mm, vias 0 -> 4
- net +5V: track 0.00 -> 177.2 mm
- net SDA1: track 0.00 -> 142.9 mm, vias 0 -> 2
- net AmpI1: track 0.00 -> 134.9 mm, vias 0 -> 2
- net SCL1: track 0.00 -> 127.3 mm
- net Amp_E1: track 0.00 -> 70.3 mm, vias 0 -> 2
- net Amp_E2: track 0.00 -> 59.2 mm
- net Vref: track 0.00 -> 50.1 mm, vias 0 -> 2
- net E1: track 0.00 -> 47.0 mm
- net +9V: track 0.00 -> 29.9 mm
- net E2: track 0.00 -> 23.5 mm
- net +3.3V: track 0.00 -> 21.7 mm
- net nó2: track 0.00 -> 21.3 mm
- net -9V: track 0.00 -> 13.2 mm
- net nó4: track 0.00 -> 9.56 mm
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
Commit message: PCB
Parts:
- removed Brd1: SSD1306, SSD1306:128x64OLED
- removed C1, C3: 1 uF, Capacitor_THT:CP_Radial_D5.0mm_P2.50mm
- removed C2, C4: 470 pF, Capacitor_THT:CP_Radial_D5.0mm_P2.50mm
- removed D1, D2, D3, D4: 1N5819, Diode_THT:D_DO-41_SOD81_P10.16mm_Horizontal
- removed J1: Vref, Connector_PinHeader_2.54mm:PinHeader_1x03_P2.54mm_Vertical
- removed J5: sinais_condicionados, Connector_PinHeader_2.54mm:PinHeader_1x04_P2.54mm_Horizontal
- removed J6: alimetacao_Master, Connector_PinHeader_2.54mm:PinHeader_1x02_P2.54mm_Vertical
- removed J7: Eletrodos, Connector_PinHeader_2.54mm:PinHeader_1x02_P2.54mm_Horizontal
- removed R1, R2, R4, R5: 100k, Resistor_THT:R_Axial_DIN0207_L6.3mm_D2.5mm_P7.62mm_Horizontal
- removed R3, R6: 220, Resistor_THT:R_Axial_DIN0207_L6.3mm_D2.5mm_P7.62mm_Horizontal
- removed R7, R8: 4k7, Resistor_THT:R_Axial_DIN0207_L6.3mm_D2.5mm_P7.62mm_Horizontal
- removed U1: AD828AN, AD828:N_8_ADI
- removed U2, U3: BluePill_STM32F103C, BluePill_breakouts:BluePill_STM32F103C
Connections:
- net AmpI2 renamed Ampl2
- net VCC renamed +12V
- net VEE renamed -12V
- J3 pad 22: AmpI1 -> Ampl1
- J4 pad 22: unconnected-(J4-Pin_22-Pad22) -> X9x10x_INC
- J4 pad 23: unconnected-(J4-Pin_23-Pad23) -> X9x10x_U/D
Routing:
- net Earth: track 214.3 -> 0.00 mm, vias 4 -> 0
- net +5V: track 177.2 -> 0.00 mm
- net SDA1: track 142.9 -> 0.00 mm, vias 2 -> 0
- net AmpI1: track 134.9 -> 0.00 mm, vias 2 -> 0
- net SCL1: track 127.3 -> 0.00 mm
- net Amp_E1: track 70.3 -> 0.00 mm, vias 2 -> 0
- net Amp_E2: track 59.2 -> 0.00 mm
- net Vref: track 50.1 -> 0.00 mm, vias 2 -> 0
- net E1: track 47.0 -> 0.00 mm
- net +9V: track 29.9 -> 0.00 mm
- net E2: track 23.5 -> 0.00 mm
- net +3.3V: track 21.7 -> 0.00 mm
- net nó2: track 21.3 -> 0.00 mm
- net -9V: track 13.2 -> 0.00 mm
- net nó4: track 9.56 -> 0.00 mm
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
Commit message: PCB
Parts:
- added Brd1: OLED, OLED_i2c:128x64OLED, F.Cu at (154.4, 155.3)
- added C1: 1 uF, Capacitor_THT:CP_Radial_D5.0mm_P2.50mm, F.Cu at (104.4, 66.5)
- added C2: 470 pF, Capacitor_THT:CP_Radial_D5.0mm_P2.50mm, F.Cu at (132.7, 74.2)
- added C3: 1 uF, Capacitor_THT:CP_Radial_D5.0mm_P2.50mm, F.Cu at (112.2, 60.2)
- added C4: 470 pF, Capacitor_THT:CP_Radial_D5.0mm_P2.50mm, F.Cu at (166.4, 53.2)
- added D1: 1N5819, Diode_THT:D_DO-41_SOD81_P10.16mm_Horizontal, F.Cu at (125.4, 78.8)
- added D2: 1N5819, Diode_THT:D_DO-41_SOD81_P10.16mm_Horizontal, F.Cu at (127.8, 93.7)
- added D3: 1N5819, Diode_THT:D_DO-41_SOD81_P10.16mm_Horizontal, F.Cu at (132.3, 50.7)
- added D4: 1N5819, Diode_THT:D_DO-41_SOD81_P10.16mm_Horizontal, F.Cu at (136.9, 59.6)
- added J1: Vref, Connector_PinHeader_2.54mm:PinHeader_1x03_P2.54mm_Vertical, F.Cu at (105.2, 82.2)
- added J5: sinais_condicionados, Connector_PinHeader_2.54mm:PinHeader_1x04_P2.54mm_Horizontal, F.Cu at (136.9, 147.1)
- added J6: Vmaster, Connector_PinHeader_2.54mm:PinHeader_1x02_P2.54mm_Vertical, F.Cu at (172.1, 145.2)
- added J7: Eletrodos, Connector_PinHeader_2.54mm:PinHeader_1x02_P2.54mm_Horizontal, F.Cu at (111.6, 52.6)
- added R1: 100k, Resistor_THT:R_Axial_DIN0207_L6.3mm_D2.5mm_P7.62mm_Horizontal, F.Cu at (109.9, 76.5)
- added R2: 100k, Resistor_THT:R_Axial_DIN0207_L6.3mm_D2.5mm_P7.62mm_Horizontal, F.Cu at (113.8, 65.2)
- added R3: 220, Resistor_THT:R_Axial_DIN0207_L6.3mm_D2.5mm_P7.62mm_Horizontal, F.Cu at (113.8, 68.7)
- added R4: 100k, Resistor_THT:R_Axial_DIN0207_L6.3mm_D2.5mm_P7.62mm_Horizontal, F.Cu at (128.7, 52.5)
- added R5: 100k, Resistor_THT:R_Axial_DIN0207_L6.3mm_D2.5mm_P7.62mm_Horizontal, F.Cu at (126.0, 56.6)
- added R6: 220, Resistor_THT:R_Axial_DIN0207_L6.3mm_D2.5mm_P7.62mm_Horizontal, F.Cu at (126.0, 60.7)
- added U1: AD828AN, AD828:N_8_ADI, F.Cu at (100.4, 55.2)
- added U2: BluePill_STM32F103C, STM32_Bluepill:BluePill_STM32F103C, F.Cu at (160.4, 103.6)
- added U3: BluePill_STM32F103C_master, STM32_Bluepill:BluePill_STM32F103C, F.Cu at (105.9, 95.3)
- added pullupscl1: 4k7, Resistor_THT:R_Axial_DIN0207_L6.3mm_D2.5mm_P7.62mm_Horizontal, F.Cu at (166.3, 127.5)
- added pullupsda1: 4k7, Resistor_THT:R_Axial_DIN0207_L6.3mm_D2.5mm_P7.62mm_Horizontal, F.Cu at (166.3, 131.5)
- moved J2 13.3 mm to (93.6, 54.9)
- moved J3 13.3 mm to (93.6, 79.0)
- moved J4 13.3 mm to (173.6, 54.9)
Connections:
- net +12V renamed VCC
- net -12V renamed VEE
- net Ampl2 renamed AmpI2
- J3 pad 22: Ampl1 -> AmpI1
- J4 pad 22: X9x10x_INC -> unconnected-(J4-Pin_22-Pad22)
- J4 pad 23: X9x10x_U/D -> unconnected-(J4-Pin_23-Pad23)
Routing:
- net Earth: track 0.00 -> 292.0 mm, vias 0 -> 4
- net Amp_E2: track 0.00 -> 191.0 mm, vias 0 -> 5
- net AmpI1: track 0.00 -> 189.6 mm, vias 0 -> 5
- net Amp_E1: track 0.00 -> 185.4 mm, vias 0 -> 8
- net +5V: track 0.00 -> 171.6 mm, vias 0 -> 2
- net SCL1: track 0.00 -> 126.0 mm, vias 0 -> 5
- net SDA1: track 0.00 -> 124.9 mm, vias 0 -> 6
- net Net-(J6-Pin_1): track 0.00 -> 90.8 mm, vias 0 -> 4
- net E1: track 0.00 -> 56.6 mm
- net Vref: track 0.00 -> 53.7 mm
- net nó4: track 0.00 -> 23.5 mm, vias 0 -> 2
- net +9V: track 0.00 -> 22.4 mm
- net E2: track 0.00 -> 18.8 mm
- net +3.3V: track 0.00 -> 17.1 mm
- net nó1: track 0.00 -> 13.6 mm
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Other:
- board text added: "+3.3V | +5.0V"

Commit message: PCB
Parts:
- moved C1 0.85 mm to (105.2, 66.5)
- moved J5 0.57 mm to (136.9, 146.5)
Routing:
- net Amp_E2: track 191.0 -> 196.1 mm
- net E2: track 18.8 -> 22.3 mm
- net nó2: track 13.1 -> 12.2 mm
- net +9V: track 22.4 -> 23.2 mm
- net Amp_E1: track 185.4 -> 184.8 mm
- net AmpI1: track 189.6 -> 189.1 mm
- net nó1: track 13.6 -> 14.1 mm

Commit message: PCB
Other:
- board text added: "Condicionamento / uC"
- board text added: "Condicionamento / uC V01 - 2023"
Changed lines of the file:
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@@
       (drillshape 0)
       (scaleselection 1)
-      (outputdirectory "gerber/drill/")
+      (outputdirectory "../gerber/drill/")
     )
   )
@@
   (gr_line (start 88.5 48.5) (end 88.5 148.4998)
     (stroke (width 0.5) (type default)) (layer "Edge.Cuts"))
+  (gr_text "Condicionamento / uC" (at 98.75 92.5 90) (layer "B.Cu")
+    (effects (font (size 1.5 1.5) (thickness 0.3) bold) (justify left bottom mirror))
+  )
+  (gr_text "Condicionamento / uC\nV01 - 2023" (at 150 119.25) (layer "B.SilkS")
+    (effects (font (size 1.5 1.5) (thickness 0.3) bold) (justify bottom))
+  )
   (gr_text "+3.3V | +5.0V" (at 102.75 79.75 90) (layer "F.SilkS")
     (effects (font (size 1.016 1.016) (thickness 0.254) bold) (justify bottom))
