File: KiCadProjects/Condicionamento/condicionamento_Aquisicao_BIA_v02/condicionamento_BIA_v02.kicad_sch (KiCad schematic)
At the start: 31 parts, among them J1 Vref, J10 nó3, J11 nó4, J2 tensoes, J3 sinais analogicos, J4 comunicacao / sinais digitais, J5 sinais_condicionados, J6 alimetacao_Master, J7 Eletrodos, J8 nó2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

Commit message: arquivos gerber para producao
Parts:
- added J12: Amp_E1, Connector_PinHeader_2.54mm:PinHeader_1x01_P2.54mm_Vertical, symbol Connector_Generic:Conn_01x01
- added J13, J16: Amp_E2, Connector_PinHeader_2.54mm:PinHeader_1x01_P2.54mm_Vertical, symbol Connector_Generic:Conn_01x01
- added J15, J17: AmpI1, Connector_PinHeader_2.54mm:PinHeader_1x01_P2.54mm_Vertical, symbol Connector_Generic:Conn_01x01
Connections:
- net AmpI1: now also J15.1 (Pin_1), J17.1 (Pin_1)
- net Amp_E1: now also J12.1 (Pin_1)
- net Amp_E2: now also J13.1 (Pin_1), J16.1 (Pin_1)
