File: KiCadProjects/Barramento_EITduino/V01/Barramento_EITduino.kicad_sch (KiCad schematic)
At the start: 3 parts, among them J2 tensoes, J3 sinais analogicos, J4 comunicacao / sinais digitais

Commit message: Primeira versao de barramento - apenas um pino de terra
Parts:
- renumbered J2 to J1, J3 to J2, J4 to J3
Changed lines of the file:
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@@
   (symbol (lib_id "Connector_Generic:Conn_01x27") (at 49.53 175.26 270) (unit 1)
     (in_bom yes) (on_board yes) (dnp no) (fields_autoplaced)
-    (property "Reference" "J3" (at 49.53 179.07 90)
+    (property "Reference" "J2" (at 49.53 179.07 90)
       (effects (font (size 1.27 1.27)) hide)
     )
@@
       (project "Barramento_EITduino"
         (path "/f0ff92cf-26e5-4ab9-977d-5f9689e8a5d0"
-          (reference "J3") (unit 1)
+          (reference "J2") (unit 1)
         )
       )
@@
   (symbol (lib_id "Connector_Generic:Conn_01x08") (at 26.035 193.04 270) (unit 1)
     (in_bom yes) (on_board yes) (dnp no)
-    (property "Reference" "J2" (at 25.4 195.58 0)
+    (property "Reference" "J1" (at 25.4 195.58 0)
       (effects (font (size 1.27 1.27)) (justify left) hide)
     )
@@
       (project "Barramento_EITduino"
         (path "/f0ff92cf-26e5-4ab9-977d-5f9689e8a5d0"
-          (reference "J2") (unit 1)
+          (reference "J1") (unit 1)
         )
       )
@@
   (symbol (lib_id "Connector_Generic:Conn_01x35") (at 131.445 192.405 270) (unit 1)
     (in_bom yes) (on_board yes) (dnp no)
-    (property "Reference" "J4" (at 131.445 196.215 90)
+    (property "Reference" "J3" (at 131.445 196.215 90)
       (effects (font (size 1.27 1.27)) hide)
     )
@@
       (project "Barramento_EITduino"
         (path "/f0ff92cf-26e5-4ab9-977d-5f9689e8a5d0"
-          (reference "J4") (unit 1)
-        )
-      )
+          (reference "J3") (unit 1)
+        )
+      )
