File: KiCadProjects/Barramento_EITduino/V03/Barramento_EITduino_V03.kicad_pcb (KiCad board)
At the start: 2 copper layers, 90 x 100 mm, 3 parts, among them J1 alimentacao analogica, J2 sinais analogicos, J3 comunicacao / sinais digitais

Commit message: novo barramento v03
Parts:
- moved J3 1.27 mm to (185.4, 57.1)
Connections:
- net CS (X9c10x) renamed CS1
- net SINC renamed SINCD
- J1 pad 1: Earth -> VCC
- J1 pad 2: VCC -> VEE
- J1 pad 3: VEE -> Earth
- J1 pad 7: -9V -> Earth
- J1 pad 8: Earth -> -9V
- J2 pad 11: unconnected-(J2-Pin_11-Pad11) -> Earth
- J2 pad 12: unconnected-(J2-Pin_12-Pad12) -> I1
- J2 pad 13: unconnected-(J2-Pin_13-Pad13) -> Earth
- J2 pad 14: Earth -> I2
- J2 pad 15: I1 -> Earth
- J2 pad 16: Earth -> Ampl1
- J2 pad 17: I2 -> Earth
- J2 pad 18: Earth -> Ampl2
- J2 pad 19: Ampl1 -> Earth
- J2 pad 20: Earth -> Sin1
- J2 pad 21: Ampl2 -> Earth
- J2 pad 22: Earth -> Sin2
- J2 pad 23: Sin1 -> Earth
- J2 pad 24: Sin2 -> SinA
- J2 pad 26: SinA -> SinB
- J2 pad 27: SinB -> Earth
- J3 pad 14: GND -> unconnected-(J3-Pin_14-Pad14)
- J3 pad 15: CS (AD9833) -> unconnected-(J3-Pin_15-Pad15)
- J3 pad 18: GND -> CS0
- J3 pad 2: Earth -> -5V
- J3 pad 3: -5V -> GND
- J3 pad 4: Earth -> GND
- J3 pad 6: Earth -> GND
- J3 pad 7: unconnected-(J3-Pin_7-Pad7) -> GND
Routing:
- net GND: track 0.00 -> 5.08 mm
- net Earth: track 0.00 -> 5.08 mm
Other:
- board text added: "CS0"
- board text added: "CS1"
- board text added: "GND"
- board text added: "SINCD"
- board text added: "SPI CIPO"
- board text added: "SPI COPI"
- board text added: "SPI clk"
- board text removed: "CS_ad9833"
- board text removed: "CS_x9c10x"
- board text removed: "DGND"
- board text removed: "SINC"
- board text removed: "SPI_CIPO"
- board text removed: "SPI_COPI"
- board text removed: "SPI_clk"
