File: KiCadProjects/Barramento_EITduino/V03/Barramento_EITduino_V03.kicad_sch (KiCad schematic)
At the start: 3 parts, among them J1 alimentacao analogica, J2 sinais analogicos, J3 comunicacao / sinais digitais

Commit message: novo barramento v03
Other:
- moved on the sheet: J1
