File: KiCadProjects/Fonte_Tensao/Fonte_tensao_LM675_v05/Fonte_tensao_LM675_v05.kicad_sch (KiCad schematic)
At the start: 33 parts, among them J1 alimentacao analogica, J2 sinais analogicos, J3 comunicacao / sinais digitais, J4 Barrel_Jack, U1 L7809, U2 LM7909_TO220, U3 LM675, U4 L7805, U5 L7905, U6 LM1117T-3.3

Commit message: fonte tensao v05
Connections:
- net VCC: no longer R1.1
- net Vin: now reaches J4.1, SW_kcd1.1
- net Vin: now also R1.1
Changed lines of the file:
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@@
   (junction (at 41.275 28.575) (diameter 0) (color 0 0 0 0)
   )
+  (junction (at 27.94 96.52) (diameter 0) (color 0 0 0 0)
+  )
   (junction (at 248.92 143.51) (diameter 0) (color 0 0 0 0)
   )
@@
     (stroke (width 0) (type default))
   )
+  (wire (pts (xy 27.94 96.52) (xy 27.94 96.266))
+    (stroke (width 0) (type default))
+  )
   (wire (pts (xy 27.94 113.03) (xy 31.75 113.03))
     (stroke (width 0) (type default))
@@
     (stroke (width 0) (type default))
   )
-  (wire (pts (xy 27.94 107.95) (xy 27.94 96.266))
-    (stroke (width 0) (type default))
-  )
   (wire (pts (xy 29.845 55.245) (xy 29.845 52.705))
     (stroke (width 0) (type default))
@@
     (stroke (width 0) (type default))
   )
+  (wire (pts (xy 22.86 132.08) (xy 22.86 137.16))
+    (stroke (width 0) (type default))
+  )
   (wire (pts (xy 80.645 38.1) (xy 80.645 40.005))
     (stroke (width 0) (type default))
@@
     (stroke (width 0) (type default))
   )
+  (wire (pts (xy 17.78 86.36) (xy 17.78 96.52))
+    (stroke (width 0) (type default))
+  )
   (wire (pts (xy 128.016 125.984) (xy 128.016 127.889))
     (stroke (width 0) (type default))
@@
     (stroke (width 0) (type default))
   )
+  (wire (pts (xy 27.94 96.52) (xy 27.94 107.95))
+    (stroke (width 0) (type default))
+  )
   (wire (pts (xy 28.575 28.575) (xy 41.275 28.575))
     (stroke (width 0) (type default))
@@
     (stroke (width 0) (type default))
   )
-  (wire (pts (xy 22.86 132.08) (xy 22.86 137.16))
-    (stroke (width 0) (type default))
-  )
   (wire (pts (xy 226.06 137.16) (xy 226.06 143.51))
     (stroke (width 0) (type default))
@@
     (stroke (width 0) (type default))
   )
+  (wire (pts (xy 17.78 96.52) (xy 27.94 96.52))
+    (stroke (width 0) (type default))
+  )
   (wire (pts (xy 49.276 136.144) (xy 53.086 136.144))
     (stroke (width 0) (type default))
@@
   (wire (pts (xy 72.771 122.174) (xy 72.771 123.444))
     (stroke (width 0) (type default))
+  )
+  (global_label "Vin" (shape input) (at 17.78 86.36 90) (fields_autoplaced)
+    (effects (font (size 1.27 1.27)) (justify left))
+    (property "Intersheetrefs" "${INTERSHEET_REFS}" (at 17.78 80.5324 90)
+      (effects (font (size 1.27 1.27)) (justify left) hide)
+    )
   )
   (global_label "SPI_clk" (shape input) (at 218.44 143.51 90) (fields_autoplaced)
@@
     (effects (font (size 1.27 1.27)) (justify left))
     (property "Intersheetrefs" "${INTERSHEET_REFS}" (at 212.09 85.4499 90)
+      (effects (font (size 1.27 1.27)) (justify left) hide)
+    )
+  )
+  (global_label "Vin" (shape input) (at 22.86 132.08 90) (fields_autoplaced)
+    (effects (font (size 1.27 1.27)) (justify left))
+    (property "Intersheetrefs" "${INTERSHEET_REFS}" (at 22.86 126.2524 90)
       (effects (font (size 1.27 1.27)) (justify left) hide)
     )
@@
         )
       )
-    )
-  )
-  (symbol (lib_name "VCC_1") (lib_id "power:VCC") (at 22.86 132.08 0) (unit 1)
-    (in_bom yes) (on_board yes) (dnp no) (fields_autoplaced)
-    (property "Reference" "#PWR017" (at 22.86 135.89 0)
-      (effects (font (size 1.27 1.27)) hide)
-    )
-    (property "Value" "VCC" (at 22.86 128.27 0)
-      (effects (font (size 1.27 1.27)))
-    )
-    (property "Footprint" "" (at 22.86 132.08 0)
-      (effects (font (size 1.27 1.27)) hide)
-    )
-    (property "Datasheet" "" (at 22.86 132.08 0)
-      (effects (font (size 1.27 1.27)) hide)
-    )
-    (pin "1")
-    (instances
-      (project "Fonte_tensao_LM675_v05"
-        (path "/f0ff92cf-26e5-4ab9-977d-5f9689e8a5d0"
-          (reference "#PWR017") (unit 1)
-        )
-      )

Commit message: versao para fabricacao jlcpcb revisao Gustavo
Parts:
- removed C6: 1uF, Capacitor_THT:CP_Radial_D5.0mm_P2.50mm, symbol Device:C_Polarized_US
- added C10: 1uF, Capacitor_THT:CP_Radial_Tantal_D4.5mm_P2.50mm, symbol Device:C_Polarized_US
- added C11: 2.2uF, Capacitor_THT:CP_Radial_Tantal_D4.5mm_P2.50mm, symbol Device:C_Polarized_US
- added C12: 100 nF, Capacitor_THT:C_Disc_D3.0mm_W1.6mm_P2.50mm, symbol Device:C_Small
- C1: value 3.3uF -> 1uF; footprint Capacitor_THT:CP_Radial_D5.0mm_P2.50mm -> Capacitor_THT:CP_Radial_Tantal_D4.5mm_P2.50mm
- C2: value 22uF -> 2.2uF; footprint Capacitor_THT:CP_Radial_D5.0mm_P2.50mm -> Capacitor_THT:CP_Radial_Tantal_D4.5mm_P2.50mm
- C3: value 1uF -> 100 nF; footprint Capacitor_THT:CP_Radial_D5.0mm_P2.50mm -> Capacitor_THT:C_Disc_D3.0mm_W1.6mm_P2.50mm; symbol Device:C_Polarized_US -> Device:C_Small
- C4, C7: footprint Capacitor_THT:CP_Radial_D5.0mm_P2.50mm -> Capacitor_THT:CP_Radial_Tantal_D4.5mm_P2.50mm
- C5: value 2.2uF -> 220nF; footprint Capacitor_THT:CP_Radial_D5.0mm_P2.50mm -> Capacitor_THT:C_Disc_D3.0mm_W1.6mm_P2.50mm; symbol Device:C_Polarized_US -> Device:C_Small
- C8: value 100uF -> 10uF; footprint Capacitor_THT:CP_Radial_D5.0mm_P2.50mm -> Capacitor_THT:CP_Radial_Tantal_D4.5mm_P2.50mm
- C9: value 100uF -> 33uF; footprint Capacitor_THT:CP_Radial_D5.0mm_P2.50mm -> Capacitor_THT:CP_Radial_Tantal_D4.5mm_P2.50mm
Connections:
- net GND is gone; now on net Earth: J3.16 (Pin_16), J3.22 (Pin_22), J3.25 (Pin_25), J3.28 (Pin_28), J3.3 (Pin_3), J3.31 (Pin_31), J3.34 (Pin_34), J3.4 (Pin_4), J3.6 (Pin_6), J3.7 (Pin_7)
- net +5V: now also C12.1
- net Earth: now also C10.2, C11.1, C12.2
- net VCC: now also C10.1
- net VEE: now also C11.2
Other:
- moved on the sheet: R3, R4, R5, R6, R7, U3
