File: KiCadProjects/Barramento_EITduino/V04/Barramento_v04.kicad_sch (KiCad schematic)
At the start: 3 parts, among them J1 alimentacao analogica, J2 sinais analogicos, J3 comunicacao / sinais digitais

Commit message: barramento utilizado na fonte de tensao V05/2023
Other:
- title: Fonte de tensao LM675 -> Barramento V04
Changed lines of the file:
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@@
   (paper "A4")
   (title_block
-    (title "Fonte de tensao LM675")
-    (date "2023-08-14")
-    (rev "v02")
+    (title "Barramento V04")
+    (date "2024-02-05")
+    (rev "v04")
     (company "EITduino")
     (comment 1 "Autor: Gustavo Pinheiro")
     (comment 2 "Barramento proposto para uma placa 90x100 mm")
-    (comment 3 "Placa face simples")
+    (comment 3 "Placa face dupla")
     (comment 4 "Pinos AGND e DGND")
     (comment 5 "capacitor 100nF ceramico")
@@
     (pin "1")
     (instances
-      (project "Fonte_tensao_LM675_v05"
+      (project "Barramento_v04"
         (path "/f0ff92cf-26e5-4ab9-977d-5f9689e8a5d0"
           (reference "#PWR015") (unit 1)
@@
     (pin "1")
     (instances
-      (project "Fonte_tensao_LM675_v05"
+      (project "Barramento_v04"
         (path "/f0ff92cf-26e5-4ab9-977d-5f9689e8a5d0"
           (reference "#PWR07") (unit 1)
@@
     (pin "1")
     (instances
-      (project "Fonte_tensao_LM675_v05"
+      (project "Barramento_v04"
         (path "/f0ff92cf-26e5-4ab9-977d-5f9689e8a5d0"
           (reference "#PWR027") (unit 1)
@@
     (pin "1")
     (instances
-      (project "Fonte_tensao_LM675_v05"
+      (project "Barramento_v04"
         (path "/f0ff92cf-26e5-4ab9-977d-5f9689e8a5d0"
           (reference "#PWR0130") (unit 1)
@@
     (pin "1")
     (instances
-      (project "Fonte_tensao_LM675_v05"
+      (project "Barramento_v04"
         (path "/f0ff92cf-26e5-4ab9-977d-5f9689e8a5d0"
           (reference "#PWR012") (unit 1)
@@
     (pin "9")
     (instances
-      (project "Fonte_tensao_LM675_v05"
+      (project "Barramento_v04"
         (path "/f0ff92cf-26e5-4ab9-977d-5f9689e8a5d0"
           (reference "J2") (unit 1)
@@
     (pin "1")
     (instances
-      (project "Fonte_tensao_LM675_v05"
+      (project "Barramento_v04"
         (path "/f0ff92cf-26e5-4ab9-977d-5f9689e8a5d0"
           (reference "#PWR0123") (unit 1)
@@
     (pin "8")
     (instances
-      (project "Fonte_tensao_LM675_v05"
+      (project "Barramento_v04"
         (path "/f0ff92cf-26e5-4ab9-977d-5f9689e8a5d0"
           (reference "J1") (unit 1)
@@
     (pin "1")
     (instances
-      (project "Fonte_tensao_LM675_v05"
+      (project "Barramento_v04"
         (path "/f0ff92cf-26e5-4ab9-977d-5f9689e8a5d0"
           (reference "#PWR06") (unit 1)
@@
     (pin "1")
     (instances
-      (project "Fonte_tensao_LM675_v05"
+      (project "Barramento_v04"
         (path "/f0ff92cf-26e5-4ab9-977d-5f9689e8a5d0"
           (reference "#PWR02") (unit 1)
@@
     (pin "1")
     (instances
-      (project "Fonte_tensao_LM675_v05"
+      (project "Barramento_v04"
         (path "/f0ff92cf-26e5-4ab9-977d-5f9689e8a5d0"
           (reference "#PWR017") (unit 1)
@@
     (pin "1")
     (instances
-      (project "Fonte_tensao_LM675_v05"
+      (project "Barramento_v04"
         (path "/f0ff92cf-26e5-4ab9-977d-5f9689e8a5d0"
           (reference "#PWR011") (unit 1)
@@
     (pin "1")
     (instances
-      (project "Fonte_tensao_LM675_v05"
+      (project "Barramento_v04"
         (path "/f0ff92cf-26e5-4ab9-977d-5f9689e8a5d0"
           (reference "#PWR026") (unit 1)
@@
     (pin "1")
     (instances
-      (project "Fonte_tensao_LM675_v05"
+      (project "Barramento_v04"
         (path "/f0ff92cf-26e5-4ab9-977d-5f9689e8a5d0"
           (reference "#PWR010") (unit 1)
@@
     (pin "1")
     (instances
-      (project "Fonte_tensao_LM675_v05"
+      (project "Barramento_v04"
         (path "/f0ff92cf-26e5-4ab9-977d-5f9689e8a5d0"
           (reference "#PWR0128") (unit 1)
@@
     (pin "1")
     (instances
-      (project "Fonte_tensao_LM675_v05"
+      (project "Barramento_v04"
         (path "/f0ff92cf-26e5-4ab9-977d-5f9689e8a5d0"
           (reference "#PWR014") (unit 1)
@@
     (pin "1")
     (instances
-      (project "Fonte_tensao_LM675_v05"
+      (project "Barramento_v04"
         (path "/f0ff92cf-26e5-4ab9-977d-5f9689e8a5d0"
           (reference "#PWR0127") (unit 1)
@@
     (pin "1")
     (instances
-      (project "Fonte_tensao_LM675_v05"
+      (project "Barramento_v04"
         (path "/f0ff92cf-26e5-4ab9-977d-5f9689e8a5d0"
           (reference "#PWR0125") (unit 1)
@@
     (pin "1")
     (instances
-      (project "Fonte_tensao_LM675_v05"
+      (project "Barramento_v04"
         (path "/f0ff92cf-26e5-4ab9-977d-5f9689e8a5d0"
           (reference "#PWR023") (unit 1)
@@
     (pin "1")
     (instances
-      (project "Fonte_tensao_LM675_v05"
+      (project "Barramento_v04"
         (path "/f0ff92cf-26e5-4ab9-977d-5f9689e8a5d0"
           (reference "#PWR0129") (unit 1)
@@
     (pin "1")
     (instances
-      (project "Fonte_tensao_LM675_v05"
+      (project "Barramento_v04"
         (path "/f0ff92cf-26e5-4ab9-977d-5f9689e8a5d0"
           (reference "#PWR04") (unit 1)
@@
     (pin "9")
     (instances
-      (project "Fonte_tensao_LM675_v05"
+      (project "Barramento_v04"
         (path "/f0ff92cf-26e5-4ab9-977d-5f9689e8a5d0"
           (reference "J3") (unit 1)
@@
     (pin "1")
     (instances
-      (project "Fonte_tensao_LM675_v05"
+      (project "Barramento_v04"
         (path "/f0ff92cf-26e5-4ab9-977d-5f9689e8a5d0"
           (reference "#PWR024") (unit 1)
@@
     (pin "1")
     (instances
-      (project "Fonte_tensao_LM675_v05"
+      (project "Barramento_v04"
         (path "/f0ff92cf-26e5-4ab9-977d-5f9689e8a5d0"
           (reference "#PWR01") (unit 1)
@@
     (pin "1")
     (instances
-      (project "Fonte_tensao_LM675_v05"
+      (project "Barramento_v04"
         (path "/f0ff92cf-26e5-4ab9-977d-5f9689e8a5d0"
           (reference "#PWR03") (unit 1)
@@
     (pin "1")
     (instances
-      (project "Fonte_tensao_LM675_v05"
+      (project "Barramento_v04"
         (path "/f0ff92cf-26e5-4ab9-977d-5f9689e8a5d0"
           (reference "#PWR025") (unit 1)
@@
     (pin "1")
     (instances
-      (project "Fonte_tensao_LM675_v05"
+      (project "Barramento_v04"
         (path "/f0ff92cf-26e5-4ab9-977d-5f9689e8a5d0"
           (reference "#PWR013") (unit 1)
@@
     (pin "1")
     (instances
-      (project "Fonte_tensao_LM675_v05"
+      (project "Barramento_v04"
         (path "/f0ff92cf-26e5-4ab9-977d-5f9689e8a5d0"
           (reference "#PWR0124") (unit 1)
@@
     (pin "1")
     (instances
-      (project "Fonte_tensao_LM675_v05"
+      (project "Barramento_v04"
         (path "/f0ff92cf-26e5-4ab9-977d-5f9689e8a5d0"
           (reference "#PWR0131") (unit 1)
@@
     (pin "1")
     (instances
-      (project "Fonte_tensao_LM675_v05"
+      (project "Barramento_v04"
         (path "/f0ff92cf-26e5-4ab9-977d-5f9689e8a5d0"
           (reference "#PWR08") (unit 1)
@@
     (pin "1")
     (instances
-      (project "Fonte_tensao_LM675_v05"
+      (project "Barramento_v04"
         (path "/f0ff92cf-26e5-4ab9-977d-5f9689e8a5d0"
           (reference "#PWR028") (unit 1)
@@
     (pin "1")
     (instances
-      (project "Fonte_tensao_LM675_v05"
+      (project "Barramento_v04"
         (path "/f0ff92cf-26e5-4ab9-977d-5f9689e8a5d0"
           (reference "#PWR016") (unit 1)
@@
     (pin "1")
     (instances
-      (project "Fonte_tensao_LM675_v05"
+      (project "Barramento_v04"
         (path "/f0ff92cf-26e5-4ab9-977d-5f9689e8a5d0"
           (reference "#PWR052") (unit 1)
@@
     (pin "1")
     (instances
-      (project "Fonte_tensao_LM675_v05"
+      (project "Barramento_v04"
         (path "/f0ff92cf-26e5-4ab9-977d-5f9689e8a5d0"
           (reference "#PWR05") (unit 1)
@@
     (pin "1")
     (instances
-      (project "Fonte_tensao_LM675_v05"
+      (project "Barramento_v04"
         (path "/f0ff92cf-26e5-4ab9-977d-5f9689e8a5d0"
           (reference "#PWR09") (unit 1)
