File: KiCadProjects/Gerador_sinais/V02/Gerador_sinais_AD9833.kicad_pcb (KiCad board)
At the start: 2 copper layers, 90 x 100 mm, 7 parts, among them J1 tensoes, J3 sinais analogicos, J4 comunicacao / sinais digitais

Commit message: versao para barramento v04
Parts:
- removed A1: Arduino_Nano_v3.x, Module:Arduino_Nano
- removed C1: 100 nF, Capacitor_THT:CP_Radial_D5.0mm_P2.50mm
- removed J1: tensoes, Connector_PinHeader_2.54mm:PinHeader_1x08_P2.54mm_Vertical
- removed J3: sinais analogicos, Connector_PinHeader_2.54mm:PinHeader_1x27_P2.54mm_Vertical
- removed J4: comunicacao / sinais digitais, Connector_PinHeader_2.54mm:PinHeader_1x35_P2.54mm_Vertical
- removed R1: 10k, Resistor_THT:R_Axial_DIN0204_L3.6mm_D1.6mm_P5.08mm_Horizontal
- removed R2: 2,7k, Resistor_THT:R_Axial_DIN0204_L3.6mm_D1.6mm_P5.08mm_Horizontal
Other:
- board outline removed
- board text removed: "+3.3V"
- board text removed: "+5V"
- board text removed: "+9V"
- board text removed: "-5V"
- board text removed: "-9V"
- board text removed: "AGND"
- board text removed: "Ampl1"
- board text removed: "Ampl2"
- board text removed: "Barramento TIE V04 2024"
- board text removed: "CS0"
- board text removed: "CS1"
- board text removed: "GND"
- board text removed: "I1"
- board text removed: "I2"
- board text removed: "SCL1"
- board text removed: "SCL2"
- board text removed: "SCL3"
- board text removed: "SCL4"
- board text removed: "SDA1"
- board text removed: "SDA2"
- board text removed: "SDA3"
- board text removed: "SDA4"
- board text removed: "SINCD"
- board text removed: "SPI_CIPO"
- board text removed: "SPI_COPI"
- board text removed: "SPI_clk"
- board text removed: "Sin1"
- board text removed: "Sin2"
- board text removed: "SinA"
- board text removed: "SinB"
- board text removed: "VCC"
- board text removed: "VEE"

Commit message: Temp
Parts:
- added A1: Arduino_Nano_v3.x, Module:Arduino_Nano, F.Cu at (-85.5, 109.8)
- added C1: 100 nF, Capacitor_THT:CP_Radial_D5.0mm_P2.50mm, F.Cu at (420.4, -39.6)
- added D1: LED - Blue, LED_THT:LED_D5.0mm, F.Cu at (134.8, -107.0)
- added D2: LED - Red, LED_THT:LED_D5.0mm, F.Cu at (142.2, -107.0)
- added D3: LED - Green, LED_THT:LED_D5.0mm, F.Cu at (-37.3, 109.0)
- added D4: LED - Yelow, LED_THT:LED_D5.0mm, F.Cu at (-29.8, 109.0)
- added J1: alimentacao analogica, Connector_PinHeader_2.54mm:PinHeader_1x08_P2.54mm_Vertical, F.Cu at (106.7, 57.1)
- added J2: sinais analogicos, Connector_PinHeader_2.54mm:PinHeader_1x27_P2.54mm_Vertical, F.Cu at (106.7, 81.3)
- added J3: comunicacao / sinais digitais, Connector_PinHeader_2.54mm:PinHeader_1x35_P2.54mm_Vertical, F.Cu at (185.4, 57.1)
- added R1: 10k, Resistor_THT:R_Axial_DIN0204_L3.6mm_D1.6mm_P5.08mm_Horizontal, F.Cu at (411.8, -41.3)
- added R2: 2,7k, Resistor_THT:R_Axial_DIN0204_L3.6mm_D1.6mm_P5.08mm_Horizontal, F.Cu at (147.8, -86.7)
- added R3: 390, Resistor_THT:R_Axial_DIN0207_L6.3mm_D2.5mm_P7.62mm_Horizontal, F.Cu at (149.9, -81.1)
- added R4: 360, Resistor_THT:R_Axial_DIN0207_L6.3mm_D2.5mm_P7.62mm_Horizontal, F.Cu at (149.9, -77.0)
- added R5: 160, Resistor_THT:R_Axial_DIN0207_L6.3mm_D2.5mm_P7.62mm_Horizontal, F.Cu at (-37.1, 142.9)
- added R6: 82, Resistor_THT:R_Axial_DIN0207_L6.3mm_D2.5mm_P7.62mm_Horizontal, F.Cu at (-37.1, 147.0)
- added SW1: botao_forma_onda, Connector_PinHeader_2.54mm:PinHeader_1x02_P2.54mm_Horizontal, F.Cu at (132.8, 146.4)
- added SW2: botao_incremento_freq, Connector_PinHeader_2.54mm:PinHeader_1x02_P2.54mm_Horizontal, F.Cu at (139.0, 146.4)
- added SW3: botao_decremento_freq, Connector_PinHeader_2.54mm:PinHeader_1x02_P2.54mm_Horizontal, F.Cu at (145.2, 146.4)
- added SW4: botao_save_Rgain, Connector_PinHeader_2.54mm:PinHeader_1x02_P2.54mm_Horizontal, F.Cu at (151.4, 146.4)
- added SW5: botao_aumenta_Rgain, Connector_PinHeader_2.54mm:PinHeader_1x02_P2.54mm_Horizontal, F.Cu at (157.6, 146.4)
- added SW6: botao_diminui_Rgain, Connector_PinHeader_2.54mm:PinHeader_1x02_P2.54mm_Horizontal, F.Cu at (163.8, 146.4)
- added U1: AD828AN, AD828:AD828, F.Cu at (148.0, -101.1)
- added U2: X9c10x, X9c10X_module:X9c10X_module, F.Cu at (140.3, -75.6)
- added U3: AD9833_module, AD9833_module:AD9833_module, F.Cu at (398.8, -52.2)
Other:
- board outline added: 90 x 100 mm
- board text added: "+3.3V"
- board text added: "+5V"
- board text added: "+9V"
- board text added: "-5V"
- board text added: "-9V"
- board text added: "AGND"
- board text added: "Ampl1"
- board text added: "Ampl2"
- board text added: "Barramento TIE V04 2024"
- board text added: "CS0"
- board text added: "CS1"
- board text added: "GND"
- board text added: "I1"
- board text added: "I2"
- board text added: "SCL1"
- board text added: "SCL2"
- board text added: "SCL3"
- board text added: "SCL4"
- board text added: "SDA1"
- board text added: "SDA2"
- board text added: "SDA3"
- board text added: "SDA4"
- board text added: "SINCD"
- board text added: "SPI_CIPO"
- board text added: "SPI_COPI"
- board text added: "SPI_clk"
- board text added: "Sin1"
- board text added: "Sin2"
- board text added: "SinA"
- board text added: "SinB"
- board text added: "VCC"
- board text added: "VEE"

Commit message: Baseado barramento v04 - Finalizado
Parts:
- removed SW1: botao_forma_onda, Connector_PinHeader_2.54mm:PinHeader_1x02_P2.54mm_Horizontal
- removed SW2: botao_incremento_freq, Connector_PinHeader_2.54mm:PinHeader_1x02_P2.54mm_Horizontal
- removed SW3: botao_decremento_freq, Connector_PinHeader_2.54mm:PinHeader_1x02_P2.54mm_Horizontal
- removed SW4: botao_save_Rgain, Connector_PinHeader_2.54mm:PinHeader_1x02_P2.54mm_Horizontal
- removed SW5: botao_aumenta_Rgain, Connector_PinHeader_2.54mm:PinHeader_1x02_P2.54mm_Horizontal
- removed SW6: botao_diminui_Rgain, Connector_PinHeader_2.54mm:PinHeader_1x02_P2.54mm_Horizontal
- added J4: Conn_01x07, Connector_PinHeader_2.54mm:PinHeader_1x07_P2.54mm_Horizontal, F.Cu at (179.8, 148.8)
- moved C1 353.1 mm to (114.0, 135.9), turned to 180 degrees
- moved R1 353.0 mm to (113.0, 146.8)
- moved U3 340.0 mm to (119.9, 142.2), turned to 90 degrees
- moved A1 261.0 mm to (175.1, 94.3), turned to 180 degrees
- moved U2 203.8 mm to (162.6, 127.0)
- moved U1 198.1 mm to (118.1, 94.7)
- moved R5 198.0 mm to (147.4, 70.9), turned to 90 degrees
- moved R2 195.9 mm to (117.9, 106.9)
- moved D3 194.4 mm to (149.5, 55.3), turned to 180 degrees
- moved R6 192.4 mm to (139.7, 71.0), turned to 90 degrees
- moved D4 180.0 mm to (142.0, 55.3), turned to 180 degrees
- moved D1 163.2 mm to (117.4, 55.3), turned to 180 degrees
- moved D2 163.2 mm to (124.9, 55.3), turned to 180 degrees
- moved R3 155.4 mm to (116.1, 70.5), turned to 90 degrees
- moved R4 150.1 mm to (123.2, 70.6), turned to 90 degrees
Routing:
- net Earth: track 0.00 -> 447.4 mm
- net SPI_COPI: track 0.00 -> 174.1 mm
- net SPI_clk: track 0.00 -> 165.4 mm
- net +5V: track 0.00 -> 159.5 mm
- net X9c10x_U/D: track 0.00 -> 108.9 mm, vias 0 -> 2
- net Out_circuito: track 0.00 -> 108.7 mm
- net CS (X9c104): track 0.00 -> 104.0 mm, vias 0 -> 2
- net CS (AD9833): track 0.00 -> 102.3 mm, vias 0 -> 3
- net S_wave: track 0.00 -> 94.1 mm
- net freq-: track 0.00 -> 88.3 mm, vias 0 -> 3
- net freq+: track 0.00 -> 86.0 mm
- net Net-(U1--IN2): track 0.00 -> 83.7 mm
- net Down_pot: track 0.00 -> 82.7 mm
- net SDA1: track 0.00 -> 80.4 mm, vias 0 -> 1
- net Up_pot: track 0.00 -> 75.8 mm
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- added copper zone on B.Cu, net Earth
- added copper zone on F.Cu, net Earth
Other:
- board text added: "Gerador Sinais V02 2024"
- board text removed: "Barramento TIE V04 2024"
