File: KiCadProjects/Gerador_sinais/V02/Gerador_sinais_AD9833.kicad_sch (KiCad schematic)
At the start: 16 parts, among them J1 tensoes, J3 sinais analogicos, J4 comunicacao / sinais digitais, SW1 botao_forma_onda, SW2 botao_incremento_freq, SW3 botao_decremento_freq, SW4 botao_save_Rgain, SW5 botao_aumenta_Rgain, SW6 botao_diminui_Rgain, U1 AD828AN, U2 X9c10x, U3 AD9833_module

Commit message: versao para barramento v04
Parts:
- SW1, SW2, SW3, SW4, SW5, SW6: footprint push_button_2_pin:SW_BUTT-2 -> Connector_PinHeader_2.54mm:PinHeader_1x02_P2.54mm_Horizontal
Changed lines of the file:
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@@
     (title "Gerador de sinais AD9833")
     (date "2023-07-12")
-    (rev "v01")
+    (rev "v02")
     (company "EITduino")
     (comment 1 "Autor: Gustavo Pinheiro")
@@
     (comment 3 "Gerador de sinais")
     (comment 4 "potenciometro digital: x9c104 (100k)")
+    (comment 5 "Baseado no barramento V04")
   )
   (junction (at 128.905 53.34) (diameter 0) (color 0 0 0 0)
@@
       (effects (font (size 1.27 1.27)) (justify left))
     )
-    (property "Footprint" "push_button_2_pin:SW_BUTT-2" (at 107.188 92.075 0)
+    (property "Footprint" "Connector_PinHeader_2.54mm:PinHeader_1x02_P2.54mm_Horizontal" (at 107.188 92.075 0)
       (effects (font (size 1.27 1.27)) hide)
     )
@@
       (effects (font (size 1.27 1.27)) (justify left))
     )
-    (property "Footprint" "push_button_2_pin:SW_BUTT-2" (at 189.357 125.603 0)
+    (property "Footprint" "Connector_PinHeader_2.54mm:PinHeader_1x02_P2.54mm_Horizontal" (at 189.357 125.603 0)
       (effects (font (size 1.27 1.27)) hide)
     )
@@
       (effects (font (size 1.27 1.27)) (justify left))
     )
-    (property "Footprint" "push_button_2_pin:SW_BUTT-2" (at 107.315 122.555 0)
+    (property "Footprint" "Connector_PinHeader_2.54mm:PinHeader_1x02_P2.54mm_Horizontal" (at 107.315 122.555 0)
       (effects (font (size 1.27 1.27)) hide)
     )
@@
       (effects (font (size 1.27 1.27)) (justify left))
     )
-    (property "Footprint" "push_button_2_pin:SW_BUTT-2" (at 107.315 107.315 0)
+    (property "Footprint" "Connector_PinHeader_2.54mm:PinHeader_1x02_P2.54mm_Horizontal" (at 107.315 107.315 0)
       (effects (font (size 1.27 1.27)) hide)
     )
@@
       (effects (font (size 1.27 1.27)) (justify left))
     )
-    (property "Footprint" "push_button_2_pin:SW_BUTT-2" (at 189.23 112.268 0)
+    (property "Footprint" "Connector_PinHeader_2.54mm:PinHeader_1x02_P2.54mm_Horizontal" (at 189.23 112.268 0)
       (effects (font (size 1.27 1.27)) hide)
     )
@@
       (effects (font (size 1.27 1.27)) (justify left))
     )
-    (property "Footprint" "push_button_2_pin:SW_BUTT-2" (at 185.928 87.63 0)
-      (effects (font (size 1.27 1.27)) hide)
-    )
+    (property "Footprint" "Connector_PinHeader_2.54mm:PinHeader_1x02_P2.54mm_Horizontal" (at 185.928 87.63 0)
+      (effects (font (size 1.27 1.27)) hide)
+    )

Commit message: mudanca do barramento para a versao V04
Parts:
- removed J1: tensoes, Connector_PinHeader_2.54mm:PinHeader_1x08_P2.54mm_Vertical, symbol Connector_Generic:Conn_01x08
- removed J3: sinais analogicos, Connector_PinHeader_2.54mm:PinHeader_1x27_P2.54mm_Vertical, symbol Connector_Generic:Conn_01x27
- removed J4: comunicacao / sinais digitais, Connector_PinHeader_2.54mm:PinHeader_1x35_P2.54mm_Vertical, symbol Connector_Generic:Conn_01x35
- added J2: sinais analogicos, Connector_PinHeader_2.54mm:PinHeader_1x27_P2.54mm_Vertical, symbol Connector_Generic:Conn_01x27
- added J5: comunicacao / sinais digitais, Connector_PinHeader_2.54mm:PinHeader_1x35_P2.54mm_Vertical, symbol Connector_Generic:Conn_01x35
- added J6: alimentacao analogica, Connector_PinHeader_2.54mm:PinHeader_1x08_P2.54mm_Vertical, symbol Connector_Generic:Conn_01x08
Connections:
- net +3.3V: now also J5.5 (Pin_5)
- net +5V: now also J5.1 (Pin_1)
- net +9V: now also J6.5 (Pin_5)
- net -5V: now also J5.2 (Pin_2)
- net -9V: now also J6.8 (Pin_8)
- net Ampl1: now also J2.16 (Pin_16)
- net Ampl2: now also J2.18 (Pin_18)
- net Earth: now also J2.11 (Pin_11), J2.13 (Pin_13), J2.15 (Pin_15), J2.17 (Pin_17), J2.19 (Pin_19), J2.21 (Pin_21), J2.23 (Pin_23), J2.25 (Pin_25), J2.27 (Pin_27), J5.16 (Pin_16), J5.22 (Pin_22), J5.25 (Pin_25), J5.28 (Pin_28), J5.3 (Pin_3), J5.31 (Pin_31), J5.34 (Pin_34), J5.4 (Pin_4), J5.6 (Pin_6), J5.7 (Pin_7), J6.3 (Pin_3), J6.4 (Pin_4), J6.6 (Pin_6), J6.7 (Pin_7)
- net I1: now also J2.12 (Pin_12)
- net I2: now also J2.14 (Pin_14)
- net Out_circuito: now also J2.24 (Pin_24)
- net Passa_alta: now also J2.20 (Pin_20)
- net SCL1: now also J5.32 (Pin_32)
- net SCL2: now also J5.29 (Pin_29)
- net SCL3: now also J5.26 (Pin_26)
- net SDA1: now also J5.33 (Pin_33)
- net SDA2: now also J5.30 (Pin_30)
- net SDA3: now also J5.27 (Pin_27)
- net SPI_CIPO: now also J5.20 (Pin_20)
- net SPI_COPI: now also J5.21 (Pin_21)
- net SPI_clk: now also J5.19 (Pin_19)
- net Sin2: now also J2.22 (Pin_22)
- net SinB: now also J2.26 (Pin_26)
- new net CS0: J5.18 (Pin_18)
- new net CS1: J5.17 (Pin_17)
- new net SCL4: J5.23 (Pin_23)
- new net SDA4: J5.24 (Pin_24)
- new net SINCD: J5.35 (Pin_35)
- new net VCC: J6.1 (Pin_1)
- new net VEE: J6.2 (Pin_2)
Other:
- moved on the sheet: SW1, SW2, SW3, SW4, SW5, SW6

Commit message: Temp
Parts:
- added D1: LED - Blue, LED_THT:LED_D5.0mm, symbol Device:LED
- added D2: LED - Red, LED_THT:LED_D5.0mm, symbol Device:LED
- added D3: LED - Green, LED_THT:LED_D5.0mm, symbol Device:LED
- added D4: LED - Yelow, LED_THT:LED_D5.0mm, symbol Device:LED
- added J4: Conn_01x06, symbol Connector_Generic:Conn_01x06
- added R3: 390, Resistor_THT:R_Axial_DIN0207_L6.3mm_D2.5mm_P7.62mm_Horizontal, symbol Device:R
- added R4: 360, Resistor_THT:R_Axial_DIN0207_L6.3mm_D2.5mm_P7.62mm_Horizontal, symbol Device:R
- added R5: 160, Resistor_THT:R_Axial_DIN0207_L6.3mm_D2.5mm_P7.62mm_Horizontal, symbol Device:R
- added R6: 82, Resistor_THT:R_Axial_DIN0207_L6.3mm_D2.5mm_P7.62mm_Horizontal, symbol Device:R
- renumbered J6 to J1, J5 to J3
Connections:
- net +3.3V: now also R6.1
- net +5V: now also R5.1
- net +9V: now also R3.1
- net -9V: now also R4.1
- net Earth: now also A1.29 (GND), D1.1 (K), D2.2 (A), D3.1 (K), D4.1 (K)
- net S_wave: now also J4.1 (Pin_1)
- new net: D4.2 (A), R6.2
- new net: D3.2 (A), R5.2
- new net: D2.1 (K), R4.2
- new net: D1.2 (A), R3.2
Other:
- moved on the sheet: A1

Commit message: Baseado barramento v04 - Finalizado
Parts:
- removed J4: Conn_01x06, symbol Connector_Generic:Conn_01x06
- removed SW1: botao_forma_onda, Connector_PinHeader_2.54mm:PinHeader_1x02_P2.54mm_Horizontal, symbol Connector_Generic:Conn_01x02
- removed SW2: botao_incremento_freq, Connector_PinHeader_2.54mm:PinHeader_1x02_P2.54mm_Horizontal, symbol Connector_Generic:Conn_01x02
- removed SW3: botao_decremento_freq, Connector_PinHeader_2.54mm:PinHeader_1x02_P2.54mm_Horizontal, symbol Connector_Generic:Conn_01x02
- removed SW4: botao_save_Rgain, Connector_PinHeader_2.54mm:PinHeader_1x02_P2.54mm_Horizontal, symbol Connector_Generic:Conn_01x02
- removed SW5: botao_aumenta_Rgain, Connector_PinHeader_2.54mm:PinHeader_1x02_P2.54mm_Horizontal, symbol Connector_Generic:Conn_01x02
- removed SW6: botao_diminui_Rgain, Connector_PinHeader_2.54mm:PinHeader_1x02_P2.54mm_Horizontal, symbol Connector_Generic:Conn_01x02
- added J4: Conn_01x07, Connector_PinHeader_2.54mm:PinHeader_1x07_P2.54mm_Horizontal, symbol Connector_Generic:Conn_01x07
Connections:
- net Down_pot: now also J4.6 (Pin_6)
- net Earth: now also J4.7 (Pin_7)
- net S_wave: now also J4.1 (Pin_1)
- net Up_pot: now also J4.5 (Pin_5)
- net freq+: now also J4.2 (Pin_2)
- net freq-: now also J4.3 (Pin_3)
- net storage_R: now also J4.4 (Pin_4)
Other:
- note added: "Selecao forma onda Incremento Freq Decremento Freq Salva Rgain Aumenta Rgain Diminui Rgain DGND"
- moved on the sheet: D1, D2, D3, D4, R3, R4, R5, R6
