File: KiCadProjects/Fonte_Corrente_Monopolar/V02/Fonte_corrente_mono_V02.kicad_pcb (KiCad board)
At the start: 2 copper layers, 90 x 100 mm, 31 parts, among them J1 alimentacao analogica, J2 sinais analogicos, J3 comunicacao / sinais digitais, J4 signal select, J7 Vref, U1-howland1 AD828AN, U2 INA128, U3-cond1 AD828AN

Commit message: Baseado barramento v04 - Finalizado - implementacao resistor pullup i2c 2
Parts:
- added RpSCL2: 4k7, Resistor_THT:R_Axial_DIN0207_L6.3mm_D2.5mm_P7.62mm_Horizontal, F.Cu at (175.2, 78.6)
- added RpSDA2: 4k7, Resistor_THT:R_Axial_DIN0207_L6.3mm_D2.5mm_P7.62mm_Horizontal, F.Cu at (179.5, 85.4)
Routing:
- net +5V: track 52.5 -> 99.7 mm
- net SCL2: track 0.00 -> 37.8 mm
- net SDA2: track 0.00 -> 29.4 mm
Changed lines of the file:
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@@
+  )
+  (footprint "Resistor_THT:R_Axial_DIN0207_L6.3mm_D2.5mm_P7.62mm_Horizontal" (layer "F.Cu")
+    (at 179.52 85.38 -90)
+    (descr "Resistor, Axial_DIN0207 series, Axial, Horizontal, pin pitch=7.62mm, 0.25W = 1/4W, length*diameter=6.3*2.5mm^2, http://cdn-reichelt.de/documents/datenblatt/B400/1_4W%23YAG.pdf")
+    (tags "Resistor Axial_DIN0207 series Axial Horizontal pin pitch 7.62mm 0.25W = 1/4W length 6.3mm diameter 2.5mm")
+    (property "Sheetfile" "Fonte_corrente_mono_V02.kicad_sch")
+    (property "Sheetname" "")
+    (property "ki_description" "Resistor")
+    (property "ki_keywords" "R res resistor")
+    (attr through_hole)
+    (fp_text reference "RpSDA2" (at 3.81 -2.37 90) (layer "F.SilkS")
+        (effects (font (size 1 1) (thickness 0.15)))
+    )
+    (fp_text value "4k7" (at 3.81 2.37 90) (layer "F.Fab")
+        (effects (font (size 1 1) (thickness 0.15)))
+    )
+    (fp_text user "${REFERENCE}" (at 3.81 0 90) (layer "F.Fab")
+        (effects (font (size 1 1) (thickness 0.15)))
+    )
+    (fp_line (start 0.54 -1.37) (end 7.08 -1.37)
+      (stroke (width 0.12) (type solid)) (layer "F.SilkS"))
+    (fp_line (start 0.54 -1.04) (end 0.54 -1.37)
+      (stroke (width 0.12) (type solid)) (layer "F.SilkS"))
+    (fp_line (start 0.54 1.04) (end 0.54 1.37)
+      (stroke (width 0.12) (type solid)) (layer "F.SilkS"))
+    (fp_line (start 0.54 1.37) (end 7.08 1.37)
+      (stroke (width 0.12) (type solid)) (layer "F.SilkS"))
+    (fp_line (start 7.08 -1.37) (end 7.08 -1.04)
+      (stroke (width 0.12) (type solid)) (layer "F.SilkS"))
+    (fp_line (start 7.08 1.37) (end 7.08 1.04)
+      (stroke (width 0.12) (type solid)) (layer "F.SilkS"))
+    (fp_line (start -1.05 -1.5) (end -1.05 1.5)
+      (stroke (width 0.05) (type solid)) (layer "F.CrtYd"))
+    (fp_line (start -1.05 1.5) (end 8.67 1.5)
+      (stroke (width 0.05) (type solid)) (layer "F.CrtYd"))
+    (fp_line (start 8.67 -1.5) (end -1.05 -1.5)
+      (stroke (width 0.05) (type solid)) (layer "F.CrtYd"))
+    (fp_line (start 8.67 1.5) (end 8.67 -1.5)
+      (stroke (width 0.05) (type solid)) (layer "F.CrtYd"))
+    (fp_line (start 0 0) (end 0.66 0)
+      (stroke (width 0.1) (type solid)) (layer "F.Fab"))
+    (fp_line (start 0.66 -1.25) (end 0.66 1.25)
+      (stroke (width 0.1) (type solid)) (layer "F.Fab"))
+    (fp_line (start 0.66 1.25) (end 6.96 1.25)
+      (stroke (width 0.1) (type solid)) (layer "F.Fab"))
+    (fp_line (start 6.96 -1.25) (end 0.66 -1.25)
+      (stroke (width 0.1) (type solid)) (layer "F.Fab"))
+    (fp_line (start 6.96 1.25) (end 6.96 -1.25)
+      (stroke (width 0.1) (type solid)) (layer "F.Fab"))
+    (fp_line (start 7.62 0) (end 6.96 0)
+      (stroke (width 0.1) (type solid)) (layer "F.Fab"))
+    (pad "1" thru_hole circle (at 0 0 270) (size 1.6 1.6) (drill 0.8) (layers "*.Cu" "*.Mask")
+      (net 5 "+5V") (pintype "passive"))
+    (pad "2" thru_hole oval (at 7.62 0 270) (size 1.6 1.6) (drill 0.8) (layers "*.Cu" "*.Mask")
+      (net 49 "SDA2") (pintype "passive"))
+    (model "${KICAD6_3DMODEL_DIR}/Resistor_THT.3dshapes/R_Axial_DIN0207_L6.3mm_D2.5mm_P7.62mm_Horizontal.wrl"
+      (offset (xyz 0 0 0))
+      (scale (xyz 1 1 1))
+      (rotate (xyz 0 0 0))
+    )
   )
   (footprint "Resistor_THT:R_Axial_DIN0207_L6.3mm_D2.5mm_P7.62mm_Horizontal" (layer "F.Cu")
@@
     )
   )
+  (footprint "Resistor_THT:R_Axial_DIN0207_L6.3mm_D2.5mm_P7.62mm_Horizontal" (layer "F.Cu")
+    (at 175.18 78.64 -90)
+    (descr "Resistor, Axial_DIN0207 series, Axial, Horizontal, pin pitch=7.62mm, 0.25W = 1/4W, length*diameter=6.3*2.5mm^2, http://cdn-reichelt.de/documents/datenblatt/B400/1_4W%23YAG.pdf")
+    (tags "Resistor Axial_DIN0207 series Axial Horizontal pin pitch 7.62mm 0.25W = 1/4W length 6.3mm diameter 2.5mm")
+    (property "Sheetfile" "Fonte_corrente_mono_V02.kicad_sch")
+    (property "Sheetname" "")
+    (property "ki_description" "Resistor")
+    (property "ki_keywords" "R res resistor")
+    (attr through_hole)
+    (fp_text reference "RpSCL2" (at 3.81 -2.37 90) (layer "F.SilkS")
+        (effects (font (size 1 1) (thickness 0.15)))
+    )
+    (fp_text value "4k7" (at 3.81 2.37 90) (layer "F.Fab")
+        (effects (font (size 1 1) (thickness 0.15)))
+    )
+    (fp_text user "${REFERENCE}" (at 3.81 0 90) (layer "F.Fab")
+        (effects (font (size 1 1) (thickness 0.15)))
+    )
+    (fp_line (start 0.54 -1.37) (end 7.08 -1.37)
+      (stroke (width 0.12) (type solid)) (layer "F.SilkS"))
+    (fp_line (start 0.54 -1.04) (end 0.54 -1.37)
+      (stroke (width 0.12) (type solid)) (layer "F.SilkS"))
+    (fp_line (start 0.54 1.04) (end 0.54 1.37)
+      (stroke (width 0.12) (type solid)) (layer "F.SilkS"))
+    (fp_line (start 0.54 1.37) (end 7.08 1.37)
+      (stroke (width 0.12) (type solid)) (layer "F.SilkS"))
+    (fp_line (start 7.08 -1.37) (end 7.08 -1.04)
+      (stroke (width 0.12) (type solid)) (layer "F.SilkS"))
+    (fp_line (start 7.08 1.37) (end 7.08 1.04)
+      (stroke (width 0.12) (type solid)) (layer "F.SilkS"))
+    (fp_line (start -1.05 -1.5) (end -1.05 1.5)
+      (stroke (width 0.05) (type solid)) (layer "F.CrtYd"))
+    (fp_line (start -1.05 1.5) (end 8.67 1.5)
+      (stroke (width 0.05) (type solid)) (layer "F.CrtYd"))
+    (fp_line (start 8.67 -1.5) (end -1.05 -1.5)
+      (stroke (width 0.05) (type solid)) (layer "F.CrtYd"))
+    (fp_line (start 8.67 1.5) (end 8.67 -1.5)
+      (stroke (width 0.05) (type solid)) (layer "F.CrtYd"))
+    (fp_line (start 0 0) (end 0.66 0)
+      (stroke (width 0.1) (type solid)) (layer "F.Fab"))
+    (fp_line (start 0.66 -1.25) (end 0.66 1.25)
+      (stroke (width 0.1) (type solid)) (layer "F.Fab"))
+    (fp_line (start 0.66 1.25) (end 6.96 1.25)
+      (stroke (width 0.1) (type solid)) (layer "F.Fab"))
+    (fp_line (start 6.96 -1.25) (end 0.66 -1.25)
+      (stroke (width 0.1) (type solid)) (layer "F.Fab"))
+    (fp_line (start 6.96 1.25) (end 6.96 -1.25)
+      (stroke (width 0.1) (type solid)) (layer "F.Fab"))
+    (fp_line (start 7.62 0) (end 6.96 0)
+      (stroke (width 0.1) (type solid)) (layer "F.Fab"))
+    (pad "1" thru_hole circle (at 0 0 270) (size 1.6 1.6) (drill 0.8) (layers "*.Cu" "*.Mask")
+      (net 5 "+5V") (pintype "passive"))
+    (pad "2" thru_hole oval (at 7.62 0 270) (size 1.6 1.6) (drill 0.8) (layers "*.Cu" "*.Mask")
+      (net 48 "SCL2") (pintype "passive"))
+    (model "${KICAD6_3DMODEL_DIR}/Resistor_THT.3dshapes/R_Axial_DIN0207_L6.3mm_D2.5mm_P7.62mm_Horizontal.wrl"
+      (offset (xyz 0 0 0))
+      (scale (xyz 1 1 1))
+      (rotate (xyz 0 0 0))
+    )
+  )
   (footprint "Capacitor_THT:CP_Radial_D5.0mm_P2.50mm" (layer "F.Cu")
     (at 164.5489 44.454)
@@
   (segment (start 125.6777 83.3976) (end 125.6777 75.6777) (width 1.27) (layer "B.Cu") (net 4))
   (segment (start 125.6777 75.6777) (end 112.484 62.484) (width 1.27) (layer "B.Cu") (net 4))
+  (segment (start 175.18 78.64) (end 183.289 70.531) (width 1.27) (layer "F.Cu") (net 5))
+  (segment (start 183.289 46.401075) (end 184.986075 44.704) (width 1.27) (layer "F.Cu") (net 5))
+  (segment (start 183.289 70.531) (end 183.289 46.401075) (width 1.27) (layer "F.Cu") (net 5))
   (segment (start 143.764 56.261) (end 145.834 56.261) (width 1.27) (layer "F.Cu") (net 5))
   (segment (start 154.58 47.515) (end 154.58 42.6) (width 1.27) (layer "F.Cu") (net 5))
+  (segment (start 184.986075 44.704) (end 185.674 44.704) (width 1.27) (layer "F.Cu") (net 5))
+  (segment (start 179.52 82.98) (end 175.18 78.64) (width 1.27) (layer "F.Cu") (net 5))
   (segment (start 145.834 56.261) (end 154.58 47.515) (width 1.27) (layer "F.Cu") (net 5))
+  (segment (start 179.52 85.38) (end 179.52 82.98) (width 1.27) (layer "F.Cu") (net 5))
   (segment (start 156.9396 42.3104) (end 156.65 42.6) (width 1.27) (layer "B.Cu") (net 5))
   (segment (start 184.8104 42.3104) (end 156.9396 42.3104) (width 1.27) (layer "B.Cu") (net 5))
@@
   (segment (start 162.584 57.064) (end 162.874 57.354) (width 1.27) (layer "B.Cu") (net 45))
   (segment (start 160.254 57.064) (end 162.584 57.064) (width 1.27) (layer "B.Cu") (net 45))
+  (segment (start 182.63 91.63) (end 182.63 115.3) (width 1.27) (layer "F.Cu") (net 48))
+  (segment (start 175.18 88.32) (end 176.3 89.44) (width 1.27) (layer "F.Cu") (net 48))
+  (segment (start 180.44 89.44) (end 182.63 91.63) (width 1.27) (layer "F.Cu") (net 48))
+  (segment (start 176.3 89.44) (end 180.44 89.44) (width 1.27) (layer "F.Cu") (net 48))
+  (segment (start 175.18 86.26) (end 175.18 88.32) (width 1.27) (layer "F.Cu") (net 48))
+  (segment (start 182.63 115.3) (end 183.154 115.824) (width 1.27) (layer "F.Cu") (net 48))
+  (segment (start 183.154 115.824) (end 185.674 115.824) (width 1.27) (layer "F.Cu") (net 48))
+  (segment (start 183.154 118.364) (end 185.674 118.364) (width 1.27) (layer "F.Cu") (net 49))
+  (segment (start 180.7 115.91) (end 183.154 118.364) (width 1.27) (layer "F.Cu") (net 49))
+  (segment (start 180.7 94.18) (end 180.7 115.91) (width 1.27) (layer "F.Cu") (net 49))
+  (segment (start 179.52 93) (end 180.7 94.18) (width 1.27) (layer "F.Cu") (net 49))
   (segment (start 128.635 113.733) (end 131.654 110.714) (width 1.27) (layer "F.Cu") (net 52))
   (segment (start 128.635 117.5) (end 128.635 113.733) (width 1.27) (layer "F.Cu") (net 52))

Commit message: Baseado barramento v04 - Finalizado
Parts:
- J7: value Vref -> +3.3V | +5.0V
- renumbered D5 to L+3.3v1, D4 to L+5v1, D6 to L+9v1, D3 to L-9v1, RganhoINA1 to Rganho-I1, Rsentinela1 to Rsentinela-I1, U2 to U2-INA-I1
Other:
- board text added: "adc_uC"

Commit message: temp
Parts:
- added RpSCL1: 4k7, Resistor_THT:R_Axial_DIN0207_L6.3mm_D2.5mm_P7.62mm_Horizontal, F.Cu at (161.0, 80.0)
- added RpSCL3: 4k7, Resistor_THT:R_Axial_DIN0207_L6.3mm_D2.5mm_P7.62mm_Horizontal, F.Cu at (167.0, 80.0)
- added RpSCL4: 4k7, Resistor_THT:R_Axial_DIN0207_L6.3mm_D2.5mm_P7.62mm_Horizontal, F.Cu at (161.0, 84.4)
- added RpSDA1: 4k7, Resistor_THT:R_Axial_DIN0207_L6.3mm_D2.5mm_P7.62mm_Horizontal, F.Cu at (173.0, 80.0)
- added RpSDA3: 4k7, Resistor_THT:R_Axial_DIN0207_L6.3mm_D2.5mm_P7.62mm_Horizontal, F.Cu at (179.0, 80.0)
- added RpSDA4: 4k7, Resistor_THT:R_Axial_DIN0207_L6.3mm_D2.5mm_P7.62mm_Horizontal, F.Cu at (173.0, 84.4)
- moved RpSCL2 21.5 mm to (154.5, 84.4)
- moved RpSDA2 12.6 mm to (167.0, 84.4)
- moved D2 4.05 mm to (167.5, 67.0)
- moved D1 1.95 mm to (177.7, 62.0)
- moved R11 1.35 mm to (164.9, 56.0)
Routing:
- net SCL1: track 0.00 -> 54.1 mm
- net SCL4: track 0.00 -> 53.6 mm
- net SDA1: track 0.00 -> 52.7 mm
- net SCL2: track 37.8 -> 79.5 mm
- net SCL3: track 0.00 -> 36.4 mm
- net +3.3V: track 58.6 -> 93.6 mm
- net SDA3: track 0.00 -> 35.0 mm
- net +5V: track 99.7 -> 127.4 mm
- net SDA4: track 0.00 -> 17.8 mm
- net SDA2: track 29.4 -> 35.6 mm
- net out_corrente: track 57.5 -> 61.3 mm, vias 0 -> 1
- net Net-(D1-K): track 43.0 -> 40.3 mm
- net +9V: track 113.0 -> 111.1 mm, vias 1 -> 0
- net nó2: track 22.3 -> 20.8 mm
- net V_INA: track 42.5 -> 41.2 mm
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Other:
- board text added: "SinA | Sin1"
