File: KiCadProjects/Demux/Demux_V01.kicad_sch (KiCad schematic)
At the start: 29 parts, among them J1 alimentacao analogica, J10 Sinais_medidos_eletrodos_16_23, J11 Sinais_medidos_eletrodos_24_31, J12 +9Vmux, J13 +5Vmux, J14 +3.3Vmux, J15 -9Vmux, J16 -5Vmux, J17 GNDmux, J18 Conn_01x03, J2 sinais analogicos, J3 comunicacao / sinais digitais, J4 Eletrodos_0_7, J5 Eletrodos_8_15, J6 Eletrodos_16_23, J7 Eletrodos_24_31, J8 Sinais_medidos_eletrodos_0_7, J9 Sinais_medidos_eletrodos_8_15, U1A1 74HC4051, U1B1 74HC4051, U2 BluePill_STM32F103C, U2A2 74HC4051, U2B2 74HC4051, U3A3 74HC4051, U3B3 74HC4051, U4A4 74HC4051, U4B4 74HC4051, U5A1 74HC4051, U5B1 74HC4051

Commit message: mudanca conectores
Parts:
- removed J10: Sinais_medidos_eletrodos_16_23, symbol Connector_Generic:Conn_01x12
- removed J11: Sinais_medidos_eletrodos_24_31, symbol Connector_Generic:Conn_01x12
- removed J4: Eletrodos_0_7, symbol Connector_Generic:Conn_01x08
- removed J5: Eletrodos_8_15, symbol Connector_Generic:Conn_01x08
- removed J6: Eletrodos_16_23, symbol Connector_Generic:Conn_01x08
- removed J7: Eletrodos_24_31, symbol Connector_Generic:Conn_01x08
- removed J8: Sinais_medidos_eletrodos_0_7, symbol Connector_Generic:Conn_01x12
- removed J9: Sinais_medidos_eletrodos_8_15, symbol Connector_Generic:Conn_01x12
- added J19, J20, J21, J22, J23, J24, J25, J26, J27, J28, J29, J30, J31, J32, J33, J34: Conn_01x06, symbol Connector_Generic:Conn_01x06
- added J4, J5, J6: Conn_01x02, symbol Connector_Generic:Conn_01x02
Connections:
- net +3.3V: now also J5.2 (Pin_2)
- net +5V: now also J4.2 (Pin_2)
- net +9V: now also J19.6 (Pin_6), J20.6 (Pin_6), J21.6 (Pin_6), J22.6 (Pin_6), J23.6 (Pin_6), J24.6 (Pin_6), J25.6 (Pin_6), J26.6 (Pin_6), J27.6 (Pin_6), J28.6 (Pin_6), J29.6 (Pin_6), J30.6 (Pin_6), J31.6 (Pin_6), J32.6 (Pin_6), J33.6 (Pin_6), J34.6 (Pin_6)
- net -9V: now also J19.5 (Pin_5), J20.5 (Pin_5), J21.5 (Pin_5), J22.5 (Pin_5), J23.5 (Pin_5), J24.5 (Pin_5), J25.5 (Pin_5), J26.5 (Pin_5), J27.5 (Pin_5), J28.5 (Pin_5), J29.5 (Pin_5), J30.5 (Pin_5), J31.5 (Pin_5), J32.5 (Pin_5), J33.5 (Pin_5), J34.5 (Pin_5)
- net E0: now also J21.2 (Pin_2)
- net E1: now also J21.1 (Pin_1)
- net E10: now also J28.1 (Pin_1)
- net E11: now also J28.2 (Pin_2)
- net E12: now also J29.1 (Pin_1)
- net E13: now also J29.2 (Pin_2)
- net E14: now also J30.1 (Pin_1)
- net E15: now also J30.2 (Pin_2)
- net E16: now also J23.1 (Pin_1)
- net E17: now also J23.2 (Pin_2)
- net E18: now also J24.1 (Pin_1)
- net E19: now also J24.2 (Pin_2)
- net E2: now also J19.1 (Pin_1)
- net E20: now also J25.1 (Pin_1)
- net E21: now also J25.2 (Pin_2)
- net E22: now also J26.1 (Pin_1)
- net E23: now also J26.2 (Pin_2)
- net E24: now also J31.1 (Pin_1)
- net E25: now also J31.2 (Pin_2)
- net E26: now also J32.1 (Pin_1)
- net E27: now also J32.2 (Pin_2)
- net E28: now also J33.1 (Pin_1)
- net E29: now also J33.2 (Pin_2)
- net E3: now also J19.2 (Pin_2)
- net E30: now also J34.1 (Pin_1)
- net E31: now also J34.2 (Pin_2)
- net E4: now also J20.1 (Pin_1)
- net E5: now also J20.2 (Pin_2)
- net E6: now also J22.1 (Pin_1)
- net E7: now also J22.2 (Pin_2)
- net E8: now also J27.1 (Pin_1)
- net E9: now also J27.2 (Pin_2)
- net Earth: now also J19.3 (Pin_3), J20.3 (Pin_3), J21.3 (Pin_3), J22.3 (Pin_3), J23.3 (Pin_3), J24.3 (Pin_3), J25.3 (Pin_3), J26.3 (Pin_3), J27.3 (Pin_3), J28.3 (Pin_3), J29.3 (Pin_3), J30.3 (Pin_3), J31.3 (Pin_3), J32.3 (Pin_3), J33.3 (Pin_3), J34.3 (Pin_3), J6.2 (Pin_2)
- new net Vref: J19.4 (Pin_4), J20.4 (Pin_4), J21.4 (Pin_4), J22.4 (Pin_4), J23.4 (Pin_4), J24.4 (Pin_4), J25.4 (Pin_4), J26.4 (Pin_4), J27.4 (Pin_4), J28.4 (Pin_4), J29.4 (Pin_4), J30.4 (Pin_4), J31.4 (Pin_4), J32.4 (Pin_4), J33.4 (Pin_4), J34.4 (Pin_4), J4.1 (Pin_1), J5.1 (Pin_1), J6.1 (Pin_1)
Other:
- note added: "A - input current"
- note added: "B - out current"
- moved on the sheet: J1, J12, J13, J14, J15, J16, J17, J18, U1A1, U1B1, U2, U2A2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
