File: KiCadProjects/Demux/V01 (cópia)/Demux_V01.kicad_pcb (KiCad board)
At the start: 2 copper layers, 90 x 100 mm, 40 parts, among them J1 alimentacao analogica, J12 +9Vmux, J13 +5Vmux, J14 +3.3Vmux, J15 -9Vmux, J16 -5Vmux, J17 GNDmux, J18 Conn_01x03, J19 Conn_01x06, J2 sinais analogicos, J20 Conn_01x06, J21 Conn_01x06, J22 Conn_01x06, J23 Conn_01x06, J24 Conn_01x06, J25 Conn_01x06, J26 Conn_01x06, J27 Conn_01x06, J28 Conn_01x06, J29 Conn_01x06, J3 comunicacao / sinais digitais, J30 Conn_01x06, J31 Conn_01x06, J32 Conn_01x06, J33 Conn_01x06, J34 Conn_01x06, J4 Conn_01x02, J5 Conn_01x02, J6 Conn_01x02, U1A1 74HC4051, U1B1 74HC4051, U2 BluePill_STM32F103C, U2A2 74HC4051, U2B2 74HC4051, U3A3 74HC4051, U3B3 74HC4051, U4A4 74HC4051, U4B4 74HC4051, U5A1 74HC4051, U5B1 74HC4051

Commit message: tmp
Parts:
- removed J16: -5Vmux, Connector_PinHeader_2.54mm:PinHeader_1x02_P2.54mm_Vertical
- removed J17: GNDmux, Connector_PinHeader_2.54mm:PinHeader_1x02_P2.54mm_Vertical
- removed J18: Conn_01x03, Connector_PinHeader_2.54mm:PinHeader_1x03_P2.54mm_Vertical
- removed J19, J20, J21, J22, J23, J24, J25, J26, J27, J28, J29, J30, J31, J32, J33, J34: Conn_01x06, Connector_PinHeader_2.54mm:PinHeader_1x06_P2.54mm_Horizontal
- added J10: +3.3Vmux, Connector_PinHeader_2.54mm:PinHeader_1x02_P2.54mm_Vertical, F.Cu at (110.2, 64.5)
- added J11: -9Vmux, Connector_PinHeader_2.54mm:PinHeader_1x02_P2.54mm_Vertical, F.Cu at (176.2, 135.2)
- added J7: Conn_01x02, Connector_PinHeader_2.54mm:PinHeader_1x02_P2.54mm_Vertical, F.Cu at (109.3, 107.2)
- added J8: +9Vmux, Connector_PinHeader_2.54mm:PinHeader_1x02_P2.54mm_Vertical, F.Cu at (110.2, 72.4)
- added J9: +5Vmux, Connector_PinHeader_2.54mm:PinHeader_1x02_P2.54mm_Vertical, F.Cu at (110.2, 68.4)
- J12: value +9Vmux -> -5Vmux
- J13: value +5Vmux -> GNDmux
- J14: value +3.3Vmux -> conectorEletrodos; footprint Connector_PinHeader_2.54mm:PinHeader_1x02_P2.54mm_Vertical -> Connector_PinHeader_2.54mm:PinHeader_2x24_P2.54mm_Vertical
- J15: value -9Vmux -> conectorEletrodos; footprint Connector_PinHeader_2.54mm:PinHeader_1x02_P2.54mm_Vertical -> Connector_PinHeader_2.54mm:PinHeader_2x24_P2.54mm_Vertical
- J4: value Conn_01x02 -> Conn_01x03; footprint Connector_PinHeader_2.54mm:PinHeader_1x02_P2.54mm_Vertical -> Connector_PinHeader_2.54mm:PinHeader_1x03_P2.54mm_Vertical
- U1A1, U1B1, U2A2, U2B2, U3A3, U3B3, U4A4, U4B4, U5A1, U5B1: footprint 74HC4051N:N16 -> HC4051:N16
- moved J14 70.6 mm to (115.5, 147.0), turned to 90 degrees
- moved U2A2 62.6 mm to (156.8, 135.9), turned to 0 degrees
- moved U4B4 57.9 mm to (164.4, 64.0), turned to 180 degrees
- moved U3B3 56.1 mm to (132.4, 64.0), turned to 180 degrees
- moved J15 50.3 mm to (115.6, 55.7), turned to 90 degrees
- moved J5 47.2 mm to (109.3, 114.5), turned to 90 degrees
- moved J6 43.6 mm to (109.3, 110.8), turned to 90 degrees
- moved U1A1 42.7 mm to (124.7, 135.9), turned to 0 degrees
- moved U4A4 42.5 mm to (149.1, 64.0), turned to 180 degrees
- moved J4 40.0 mm to (174.3, 89.3), turned to 90 degrees
- moved J12 35.9 mm to (176.2, 131.2), turned to 90 degrees
- moved J13 35.1 mm to (176.2, 127.2), turned to 90 degrees
- moved U5B1 34.1 mm to (180.3, 111.4), turned to 0 degrees
- moved U2B2 34.1 mm to (172.0, 135.9), turned to 0 degrees
- moved U2 33.1 mm to (168.8, 92.7), turned to -90 degrees
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Connections:
- J12 pad 1: VCC_DEMUX -> VEE_DEMUX
- J12 pad 2: +9V -> -5V
- J13 pad 1: VCC_DEMUX -> VEE_DEMUX
- J13 pad 2: +5V -> Earth
- J14 pad 1: VCC_DEMUX -> E0
- J14 pad 2: +3.3V -> E1
- J15 pad 1: VEE_DEMUX -> E16
- J15 pad 2: -9V -> E17
- J3 pad 13: unconnected-(J3-Pin_13-Pad13) -> SINC_C
- J3 pad 14: unconnected-(J3-Pin_14-Pad14) -> SINC_B
- J3 pad 15: unconnected-(J3-Pin_15-Pad15) -> SINC_A
- J4 pad 1: Vref -> I2
- J4 pad 2: +5V -> In_B
- J5 pad 2: +3.3V -> +5V
- J6 pad 2: Earth -> +3.3V
- U1A1 pad 10: S1 -> A_S1
- U1A1 pad 11: S0 -> A_S0
- U1A1 pad 3: DEMUX1 -> DEMUXA1
- U1A1 pad 9: S2 -> A_S2
- U1B1 pad 10: S1 -> B_S1
- U1B1 pad 11: S0 -> B_S0
- U1B1 pad 3: DEMUX1B -> DEMUXB1
- U1B1 pad 9: S2 -> B_S2
- U2 pad 10: unconnected-(U2-PA5_SCK1-Pad10) -> SINC_A
- U2 pad 11: unconnected-(U2-PA6_MISO1-Pad11) -> SINC_B
- U2 pad 12: unconnected-(U2-PA7_MOSI1-Pad12) -> SINC_C
- U2 pad 14: Enable_A4 -> Enable_B2
- U2 pad 15: unconnected-(U2-PB10_SCL2-Pad15) -> Enable_B3
- U2 pad 16: unconnected-(U2-PB11_SDA2-Pad16) -> Enable_B4
- U2 pad 21: S0 -> B_S3
- U2 pad 22: unconnected-(U2-PB13_SCK2-Pad22) -> B_S2
- U2 pad 23: unconnected-(U2-PB14_MISO2-Pad23) -> B_S1
- U2 pad 24: unconnected-(U2-PB15_MOSI2-Pad24) -> B_S0
- U2 pad 25: S1 -> unconnected-(U2-PA8-Pad25)
- U2 pad 3: unconnected-(U2-PC14-Pad3) -> SINCD
- U2 pad 30: S2 -> A_S3
- U2 pad 31: S3 -> A_S2
- U2 pad 32: S4 -> A_S1
- U2 pad 33: Enable_A1 -> A_S0
- U2 pad 34: unconnected-(U2-PB6_SCL1-Pad34) -> SCL1
- U2 pad 35: unconnected-(U2-PB7_SDA1-Pad35) -> SDA1
- U2 pad 36: Enable_A2 -> B_S4
- U2 pad 37: Enable_A3 -> A_S4
- U2 pad 4: unconnected-(U2-PC15-Pad4) -> Enable_A1
- U2 pad 5: Enable_B4 -> Enable_A2
- U2 pad 6: Enable_B3 -> Enable_A3
- U2 pad 7: unconnected-(U2-PA2_TX2-Pad7) -> Enable_A4
- U2 pad 9: Enable_B2 -> unconnected-(U2-PA4-Pad9)
- U2A2 pad 10: S1 -> A_S1
- U2A2 pad 11: S0 -> A_S0
- U2A2 pad 3: DEMUX2A -> DEMUXA2
- U2A2 pad 9: S2 -> A_S2
- U2B2 pad 10: S1 -> SB1
- U2B2 pad 11: S0 -> SB0
- U2B2 pad 3: DEMUX2B -> DEMUXB2
- U2B2 pad 9: S2 -> SB2
- U3A3 pad 3: DEMUX3A -> DEMUXA3
- U3B3 pad 3: DEMUX3B -> DEMUXB3
- U4A4 pad 3: DEMUX4A -> DEMUXA4
- U4B4 pad 3: DEMUX4B -> DEMUXB4
- U5A1 pad 10: S4 -> A_S4
- U5A1 pad 11: S3 -> A_S3
- U5A1 pad 6: Earth -> Enable_A
- U5B1 pad 10: S4 -> B_S4
- U5B1 pad 11: S3 -> B_S3
- U5B1 pad 6: Earth -> Enable_B
Routing:
- net -9V: track 373.3 -> 0.00 mm, vias 1 -> 0
- net Vref: track 354.1 -> 0.00 mm
- net +9V: track 353.6 -> 0.00 mm, vias 1 -> 0
- net VEE_DEMUX: track 197.6 -> 0.00 mm, vias 2 -> 0
- net S1: track 171.6 -> 0.00 mm, vias 6 -> 0
- net S0: track 164.8 -> 0.00 mm, vias 7 -> 0
- net E29: track 162.7 -> 0.00 mm, vias 5 -> 0
- net VCC_DEMUX: track 159.5 -> 0.00 mm, vias 3 -> 0
- net S2: track 152.7 -> 0.00 mm, vias 4 -> 0
- net +5V: track 149.3 -> 0.00 mm, vias 6 -> 0
- net E11: track 115.0 -> 0.00 mm, vias 5 -> 0
- net E6: track 112.3 -> 0.00 mm, vias 5 -> 0
- net E12: track 106.9 -> 0.00 mm, vias 2 -> 0
- net E2: track 103.8 -> 0.00 mm, vias 1 -> 0
- net E24: track 98.5 -> 0.00 mm, vias 5 -> 0
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
Commit message: tmp
Parts:
- U1A1, U1B1, U2A2, U2B2, U3A3, U3B3, U4A4, U4B4, U5A1, U5B1: footprint HC4051:N16 -> 74HC4051N:N16
- moved J5 77.0 mm to (176.0, 75.8), turned to -90 degrees
- moved J6 73.7 mm to (176.0, 79.4), turned to -90 degrees
- moved J7 70.9 mm to (176.0, 83.0), turned to -90 degrees
- moved J4 68.7 mm to (110.0, 113.5), turned to 180 degrees
- moved J8 66.8 mm to (176.0, 61.0), turned to -90 degrees
- moved J11 66.4 mm to (110.0, 130.0)
- moved J12 66.4 mm to (110.0, 126.0)
- moved J13 66.4 mm to (110.0, 122.0)
- moved J10 66.0 mm to (176.0, 68.9), turned to -90 degrees
- moved J9 65.9 mm to (176.0, 65.0), turned to -90 degrees
- moved U5A1 35.5 mm to (110.4, 68.8), turned to 180 degrees
- moved U3A3 33.5 mm to (142.0, 86.4), turned to 0 degrees
- moved U1B1 28.0 mm to (118.0, 118.6), turned to 180 degrees
- moved U5B1 24.9 mm to (178.6, 136.2)
- moved U4B4 22.7 mm to (168.0, 86.4), turned to 0 degrees
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Connections:
- J14 pad 13: E4 -> E8
- J14 pad 14: E5 -> E9
- J14 pad 19: E6 -> E12
- J14 pad 20: E7 -> E13
- J14 pad 25: E8 -> E2
- J14 pad 26: E9 -> E3
- J14 pad 31: E10 -> E6
- J14 pad 32: E11 -> E7
- J14 pad 37: E12 -> E10
- J14 pad 38: E13 -> E11
- J14 pad 7: E2 -> E4
- J14 pad 8: E3 -> E5
- J15 pad 13: E20 -> E24
- J15 pad 14: E21 -> E25
- J15 pad 19: E22 -> E28
- J15 pad 20: E23 -> E29
- J15 pad 25: E24 -> E18
- J15 pad 26: E25 -> E19
- J15 pad 31: E26 -> E22
- J15 pad 32: E27 -> E23
- J15 pad 37: E28 -> E26
- J15 pad 38: E29 -> E27
- J15 pad 7: E18 -> E20
- J15 pad 8: E19 -> E21
Routing:
- net Earth: track 0.00 -> 318.1 mm, vias 0 -> 21
- net +9V: track 0.00 -> 261.2 mm
- net -9V: track 0.00 -> 260.3 mm
- net Vref: track 0.00 -> 220.4 mm
- net VCC_DEMUX: track 0.00 -> 217.8 mm, vias 0 -> 1
- net VEE_DEMUX: track 0.00 -> 193.6 mm, vias 0 -> 1
- net -5V: track 0.00 -> 159.0 mm, vias 0 -> 1
- net DEMUXB3: track 0.00 -> 88.0 mm
- net DEMUXA2: track 0.00 -> 85.5 mm
- net DEMUXA1: track 0.00 -> 75.6 mm, vias 0 -> 1
- net B_S3: track 0.00 -> 74.2 mm
- net A_S4: track 0.00 -> 73.3 mm
- net In_B: track 0.00 -> 66.2 mm
- net DEMUXB4: track 0.00 -> 63.9 mm
- net E31: track 0.00 -> 63.6 mm
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Other:
- board text added: "---"
- board text added: "16 - CANAIS"
- board text added: "Select Iout"
- board text added: "VCC - DEMUX"
- board text added: "VEE - Demux"
- board text added: "Vref - canais"
