File: KiCadProjects/Demux/V01 (cópia)/Demux_V01.kicad_sch (KiCad schematic)
At the start: 28 parts, among them J1 alimentacao analogica, J12 +9Vmux, J13 +5Vmux, J14 +3.3Vmux, J15 -9Vmux, J16 -5Vmux, J17 GNDmux, J18 Conn_01x03, J19 Conn_01x06, J2 sinais analogicos, J20 Conn_01x06, J21 Conn_01x06, J22 Conn_01x06, J27 Conn_01x06, J28 Conn_01x06, J29 Conn_01x06, J3 comunicacao / sinais digitais, J30 Conn_01x06, J4 Conn_01x02, J5 Conn_01x02, J6 Conn_01x02, U1A1 74HC4051, U1B1 74HC4051, U2 BluePill_STM32F103C, U2A2 74HC4051, U2B2 74HC4051, U5A1 74HC4051, U5B1 74HC4051

Commit message: tmp
Parts:
- removed J19, J20, J21, J22, J27, J28, J29, J30: Conn_01x06, Connector_PinHeader_2.54mm:PinHeader_1x06_P2.54mm_Horizontal, symbol Connector_Generic:Conn_01x06
- added J14, J15: conectorEletrodos, Connector_PinHeader_2.54mm:PinHeader_2x24_P2.54mm_Vertical, symbol Connector_Generic:Conn_02x24_Top_Bottom
- added U3A3, U3B3, U4A4, U4B4: 74HC4051, HC4051:N16, symbol 74xx:74HC4051
- U1A1, U1B1, U2A2, U2B2, U5A1, U5B1: footprint 74HC4051N:N16 -> HC4051:N16
- renumbered J14 to J10, J15 to J11, J16 to J12, J17 to J13, J18 to J4, J4 to J5, J5 to J6, J6 to J7, J12 to J8, J13 to J9
Connections:
- net +9V: now also J14.12 (Pin_12), J14.18 (Pin_18), J14.24 (Pin_24), J14.30 (Pin_30), J14.36 (Pin_36), J14.42 (Pin_42), J14.48 (Pin_48), J14.6 (Pin_6), J15.12 (Pin_12), J15.18 (Pin_18), J15.24 (Pin_24), J15.30 (Pin_30), J15.36 (Pin_36), J15.42 (Pin_42), J15.48 (Pin_48), J15.6 (Pin_6)
- net -9V: now also J14.11 (Pin_11), J14.17 (Pin_17), J14.23 (Pin_23), J14.29 (Pin_29), J14.35 (Pin_35), J14.41 (Pin_41), J14.47 (Pin_47), J14.5 (Pin_5), J15.11 (Pin_11), J15.17 (Pin_17), J15.23 (Pin_23), J15.29 (Pin_29), J15.35 (Pin_35), J15.41 (Pin_41), J15.47 (Pin_47), J15.5 (Pin_5)
- net E0: now also J14.1 (Pin_1)
- net E1: now also J14.2 (Pin_2)
- net E10: now also J14.31 (Pin_31)
- net E11: now also J14.32 (Pin_32)
- net E12: now also J14.37 (Pin_37)
- net E13: now also J14.38 (Pin_38)
- net E14: now also J14.43 (Pin_43)
- net E15: now also J14.44 (Pin_44)
- net E2: now also J14.7 (Pin_7)
- net E3: now also J14.8 (Pin_8)
- net E4: now also J14.13 (Pin_13)
- net E5: now also J14.14 (Pin_14)
- net E6: now also J14.19 (Pin_19)
- net E7: now also J14.20 (Pin_20)
- net E8: now also J14.25 (Pin_25)
- net E9: now also J14.26 (Pin_26)
- net Earth: now also J14.15 (Pin_15), J14.21 (Pin_21), J14.27 (Pin_27), J14.3 (Pin_3), J14.33 (Pin_33), J14.39 (Pin_39), J14.45 (Pin_45), J14.9 (Pin_9), J15.15 (Pin_15), J15.21 (Pin_21), J15.27 (Pin_27), J15.3 (Pin_3), J15.33 (Pin_33), J15.39 (Pin_39), J15.45 (Pin_45), J15.9 (Pin_9), U3A3.8 (GND), U3B3.8 (GND), U4A4.8 (GND), U4B4.8 (GND); no longer U5A1.10 (S1), U5B1.10 (S1)
- net Enable_B1: now also U2.13 (PB0); no longer U2.6 (PA1)
- net Enable_B2: now also U2.14 (PB1); no longer U2.7 (PA2_TX2)
- net VCC_DEMUX: now also U3A3.16 (VCC), U3B3.16 (VCC), U4A4.16 (VCC), U4B4.16 (VCC)
- net VEE_DEMUX: now also U3A3.7 (VEE), U3B3.7 (VEE), U4A4.7 (VEE), U4B4.7 (VEE)
- net Vref: now also J14.10 (Pin_10), J14.16 (Pin_16), J14.22 (Pin_22), J14.28 (Pin_28), J14.34 (Pin_34), J14.4 (Pin_4), J14.40 (Pin_40), J14.46 (Pin_46), J15.10 (Pin_10), J15.16 (Pin_16), J15.22 (Pin_22), J15.28 (Pin_28), J15.34 (Pin_34), J15.4 (Pin_4), J15.40 (Pin_40), J15.46 (Pin_46)
- net DEMUXA4: now reaches U5A1.12 (A3)
- net DEMUXA4: now also U4A4.3 (A)
- net DEMUXA3: now reaches U5A1.15 (A2)
- net DEMUXA3: now also U3A3.3 (A)
- net DEMUXB4: now reaches U5B1.12 (A3)
- net DEMUXB4: now also U4B4.3 (A)
- net DEMUXB3: now reaches U5B1.15 (A2)
- net DEMUXB3: now also U3B3.3 (A)
- net Enable_B3: now reaches U2.15 (PB10_SCL2)
- net Enable_B3: now also U3B3.6 (~{E})
- net Enable_B4: now reaches U2.16 (PB11_SDA2)
- net Enable_B4: now also U4B4.6 (~{E})
- net B_S4: now reaches U2.36 (PB8)
- net B_S4: now also U5B1.10 (S1)
- net A_S4: now reaches U2.37 (PB9)
- net A_S4: now also U5A1.10 (S1)
- new net E16: J15.1 (Pin_1), U3A3.13 (A0), U3B3.13 (A0)
- new net E17: J15.2 (Pin_2), U3A3.14 (A1), U3B3.14 (A1)
- new net E18: J15.7 (Pin_7), U3A3.15 (A2), U3B3.15 (A2)
- new net E19: J15.8 (Pin_8), U3A3.12 (A3), U3B3.12 (A3)
- new net E20: J15.13 (Pin_13), U3A3.1 (A4), U3B3.1 (A4)
- new net E21: J15.14 (Pin_14), U3A3.5 (A5), U3B3.5 (A5)
- new net E22: J15.19 (Pin_19), U3A3.2 (A6), U3B3.2 (A6)
- new net E23: J15.20 (Pin_20), U3A3.4 (A7), U3B3.4 (A7)
- new net E24: J15.25 (Pin_25), U4A4.13 (A0), U4B4.13 (A0)
- new net E25: J15.26 (Pin_26), U4A4.14 (A1), U4B4.14 (A1)
- new net E26: J15.31 (Pin_31), U4A4.15 (A2), U4B4.15 (A2)
- new net E27: J15.32 (Pin_32), U4A4.12 (A3), U4B4.12 (A3)
- new net E28: J15.37 (Pin_37), U4A4.1 (A4), U4B4.1 (A4)
- new net E29: J15.38 (Pin_38), U4A4.5 (A5), U4B4.5 (A5)
- new net E30: J15.43 (Pin_43), U4A4.2 (A6), U4B4.2 (A6)
- new net E31: J15.44 (Pin_44), U4A4.4 (A7), U4B4.4 (A7)
- new net Enable_A3: U2.6 (PA1), U3A3.6 (~{E})
- new net Enable_A4: U2.7 (PA2_TX2), U4A4.6 (~{E})
- new net S0: U3A3.11 (S0), U3B3.11 (S0), U4A4.11 (S0), U4B4.11 (S0)
- new net S1: U3A3.10 (S1), U3B3.10 (S1), U4A4.10 (S1), U4B4.10 (S1)
- new net S2: U3A3.9 (S2), U3B3.9 (S2), U4A4.9 (S2), U4B4.9 (S2)
Other:
- company: EITduino -> Autor: Gustavo Pinheiro
- title: Barramento V04 -> Demux
- moved on the sheet: J1, J4, U1B1, U2A2, U2B2, U5B1

Commit message: tmp
Parts:
- U1A1, U1B1, U2A2, U2B2, U3A3, U3B3, U4A4, U4B4, U5A1, U5B1: footprint HC4051:N16 -> 74HC4051N:N16
Connections:
- net E10: now also J14.37 (Pin_37); no longer J14.31 (Pin_31)
- net E11: now also J14.38 (Pin_38); no longer J14.32 (Pin_32)
- net E12: now also J14.19 (Pin_19); no longer J14.37 (Pin_37)
- net E13: now also J14.20 (Pin_20); no longer J14.38 (Pin_38)
- net E18: now also J15.25 (Pin_25); no longer J15.7 (Pin_7)
- net E19: now also J15.26 (Pin_26); no longer J15.8 (Pin_8)
- net E2: now also J14.25 (Pin_25); no longer J14.7 (Pin_7)
- net E20: now also J15.7 (Pin_7); no longer J15.13 (Pin_13)
- net E21: now also J15.8 (Pin_8); no longer J15.14 (Pin_14)
- net E22: now also J15.31 (Pin_31); no longer J15.19 (Pin_19)
- net E23: now also J15.32 (Pin_32); no longer J15.20 (Pin_20)
- net E24: now also J15.13 (Pin_13); no longer J15.25 (Pin_25)
- net E25: now also J15.14 (Pin_14); no longer J15.26 (Pin_26)
- net E26: now also J15.37 (Pin_37); no longer J15.31 (Pin_31)
- net E27: now also J15.38 (Pin_38); no longer J15.32 (Pin_32)
- net E28: now also J15.19 (Pin_19); no longer J15.37 (Pin_37)
- net E29: now also J15.20 (Pin_20); no longer J15.38 (Pin_38)
- net E3: now also J14.26 (Pin_26); no longer J14.8 (Pin_8)
- net E4: now also J14.7 (Pin_7); no longer J14.13 (Pin_13)
- net E5: now also J14.8 (Pin_8); no longer J14.14 (Pin_14)
- net E6: now also J14.31 (Pin_31); no longer J14.19 (Pin_19)
- net E7: now also J14.32 (Pin_32); no longer J14.20 (Pin_20)
- net E8: now also J14.13 (Pin_13); no longer J14.25 (Pin_25)
- net E9: now also J14.14 (Pin_14); no longer J14.26 (Pin_26)
Other:
- moved on the sheet: J14, J15
