File: KiCadProjects/Demux/V02/Demux_V02.kicad_sch (KiCad schematic)
At the start: 26 parts, among them J1 alimentacao analogica, J10 +3.3Vmux, J11 -9Vmux, J12 -5Vmux, J13 GNDmux, J14 conectorEletrodos, J15 conectorEletrodos, J2 sinais analogicos, J3 comunicacao / sinais digitais, J4 Conn_01x03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

Commit message: para producao
Connections:
- net Enable_A: now also U2.9 (PA4)
- net Enable_B: now also U2.25 (PA8)
- net SINCD: now also U2.8 (PA3_RX2); no longer U2.3 (PC14)

Commit message: tmp
Parts:
- added L+3.3v1: LED Yelow, LED_THT:LED_D5.0mm, symbol Device:LED
- added L+5v1: LED Green, LED_THT:LED_D5.0mm, symbol Device:LED
- added L+9v1: LED Blue, LED_THT:LED_D5.0mm, symbol Device:LED
- added L-9v1: LED Red, LED_THT:LED_D5.0mm, symbol Device:LED
- added R1, R2: 1.5k, Resistor_THT:R_Axial_DIN0207_L6.3mm_D2.5mm_P7.62mm_Horizontal, symbol Device:R
- added R3: 470, Resistor_THT:R_Axial_DIN0207_L6.3mm_D2.5mm_P7.62mm_Horizontal, symbol Device:R
- added R4: 510, Resistor_THT:R_Axial_DIN0207_L6.3mm_D2.5mm_P7.62mm_Horizontal, symbol Device:R
Connections:
- net +3.3V: now also R4.1
- net +5V: now also R3.1
- net +9V: now also R1.1
- net -9V: now also R2.1
- net Earth: now also L+3.3v1.1 (K), L+5v1.1 (K), L+9v1.1 (K), L-9v1.2 (A)
- new net: L-9v1.1 (K), R2.2
- new net: L+3.3v1.2 (A), R4.2
- new net: L+9v1.2 (A), R1.2
- new net: L+5v1.2 (A), R3.2
