File: KiCadProjects/Aquisicao/Aquisicao_STM_barramento_V01/Aquisicao_STM_Barramento_v01.kicad_pcb (KiCad board)
At the start: 2 copper layers, 90 x 100 mm, 3 parts, among them J1 alimentacao analogica, J2 sinais analogicos, J3 comunicacao / sinais digitais

Commit message: tmp
Parts:
- added C1: 680u, Capacitor_THT:CP_Radial_D5.0mm_P2.50mm, F.Cu at (157.7, 147.3)
- added C2: 220u, Capacitor_THT:CP_Radial_D5.0mm_P2.50mm, F.Cu at (151.3, 145.6)
- added C3: 10uF, Capacitor_THT:CP_Radial_Tantal_D4.5mm_P2.50mm, F.Cu at (169.1, 141.5)
- added C4: 33uF, Capacitor_THT:CP_Radial_Tantal_D4.5mm_P2.50mm, F.Cu at (175.6, 141.8)
- added D1: 1N5819, Diode_THT:D_DO-41_SOD81_P10.16mm_Horizontal, F.Cu at (151.9, 142.0)
- added J4: Conn_01x04, Connector_PinHeader_2.54mm:PinHeader_1x04_P2.54mm_Horizontal, F.Cu at (122.3, 146.7)
- added L1: 33u, Inductor_SMD:L_7.3x7.3_H4.5, F.Cu at (144.4, 142.7)
- added U1: BluePill_STM32F103C, BluePill_STM32:BluePill_STM32F103C, F.Cu at (177.9, 103.7)
- added U2: LM2596S-5, Package_TO_SOT_THT:TO-220-5_P3.4x3.7mm_StaggerOdd_Lead3.8mm_Vertical, F.Cu at (137.9, 141.8)
- added U3: LM1117T-3.3, Package_TO_SOT_THT:TO-220-3_Vertical, F.Cu at (172.0, 146.7)
- added U4: BluePill_STM32F103C, BluePill_STM32:BluePill_STM32F103C, F.Cu at (129.4, 103.7)
- added U5: BluePill_STM32F103C, BluePill_STM32:BluePill_STM32F103C, F.Cu at (153.6, 103.7)
- added U6: BluePill_STM32F103C, BluePill_STM32:BluePill_STM32F103C, F.Cu at (171.9, 118.4)
Connections:
- J3 pad 13: unconnected-(J3-Pin_13-Pad13) -> SINC_C
- J3 pad 14: unconnected-(J3-Pin_14-Pad14) -> SINC_B
- J3 pad 15: unconnected-(J3-Pin_15-Pad15) -> SINC_A
Routing:
- net SCL1: track 0.00 -> 224.6 mm, vias 0 -> 2
- net SINC_A: track 0.00 -> 224.2 mm
- net SINC_B: track 0.00 -> 216.9 mm, vias 0 -> 1
- net SINCD: track 0.00 -> 203.6 mm, vias 0 -> 2
- net Ampl2: track 0.00 -> 186.7 mm
- net SDA1: track 0.00 -> 182.1 mm
- net SINC_C: track 0.00 -> 175.7 mm
- net Ampl1: track 0.00 -> 163.6 mm, vias 0 -> 2
- net VCC: track 0.00 -> 160.5 mm
- net 3.3V_step: track 0.00 -> 116.5 mm, vias 0 -> 1
- net sign_C1: track 0.00 -> 106.2 mm
- net sign_C3: track 0.00 -> 74.5 mm, vias 0 -> 1
- net sign_C2: track 0.00 -> 65.9 mm
- net sign_C4: track 0.00 -> 62.3 mm
- net 5V_stepdown: track 0.00 -> 50.4 mm
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- added copper zone on B.Cu, net Earth
- added copper zone on F.Cu, net Earth
Other:
- board text added: "Aquisicao V01 2024"
- board text added: "STM32-C1"
- board text added: "STM32-C2"
- board text added: "STM32-C3"
- board text added: "STM32-C4"
- board text removed: "Barramento TIE V04 2024"

Commit message: para producao
Parts:
- added J5: Conn_01x04, Connector_PinHeader_2.54mm:PinHeader_1x04_P2.54mm_Horizontal, F.Cu at (181.1, 146.6)
- moved C4 8.14 mm to (167.5, 141.2)
- moved C1 5.18 mm to (152.6, 146.8)
- moved D1 5.15 mm to (146.8, 141.8)
- moved U2 5.15 mm to (132.7, 141.7)
- moved U3 5.15 mm to (166.9, 146.6)
- moved C2 5.15 mm to (146.2, 145.5)
- moved C3 5.15 mm to (164.0, 141.4)
- moved L1 5.15 mm to (139.2, 142.5)
- moved J4 1.48 mm to (120.9, 146.7)
Connections:
- U1 pad 13: unconnected-(U1-PB0-Pad13) -> sign_C5
- U1 pad 14: unconnected-(U1-PB1-Pad14) -> SINCD
- U1 pad 3: SINCD -> unconnected-(U1-PC14-Pad3)
- U4 pad 13: unconnected-(U4-PB0-Pad13) -> sign_C6
- U4 pad 14: unconnected-(U4-PB1-Pad14) -> SINCD
- U4 pad 3: SINCD -> unconnected-(U4-PC14-Pad3)
- U5 pad 13: unconnected-(U5-PB0-Pad13) -> sign_C7
- U5 pad 14: unconnected-(U5-PB1-Pad14) -> SINCD
- U5 pad 3: SINCD -> unconnected-(U5-PC14-Pad3)
- U6 pad 13: unconnected-(U6-PB0-Pad13) -> sign_C8
- U6 pad 14: unconnected-(U6-PB1-Pad14) -> SINCD
- U6 pad 3: SINCD -> unconnected-(U6-PC14-Pad3)
Routing:
- net Earth: track 0.00 -> 388.8 mm, vias 9 -> 20
- net sign_C6: track 0.00 -> 126.4 mm
- net sign_C5: track 0.00 -> 87.7 mm
- net sign_C7: track 0.00 -> 84.9 mm
- net sign_C8: track 0.00 -> 57.7 mm, vias 0 -> 1
- net SINC_B: track 216.9 -> 162.8 mm, vias 1 -> 2
- net SCL1: track 224.6 -> 178.7 mm, vias 2 -> 1
- net SINC_A: track 224.2 -> 181.2 mm
- net SINCD: track 203.6 -> 225.6 mm, vias 2 -> 0
- net Ampl2: track 186.7 -> 207.3 mm
- net sign_C3: track 74.5 -> 86.0 mm, vias 1 -> 2
- net VCC: track 160.5 -> 151.7 mm
- net SDA1: track 182.1 -> 173.5 mm, vias 0 -> 1
- net sign_C2: track 65.9 -> 59.9 mm
- net sign_C1: track 106.2 -> 111.5 mm
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Other:
- board text added: "C1"
- board text added: "C2"
- board text added: "C3"
- board text added: "C4"
- board text added: "C5"
- board text added: "C6"
- board text added: "C7"
- board text added: "C8"
- board text added: "STM32-C1/C5"
- board text added: "STM32-C2/C6"
- board text added: "STM32-C3/C7"
- board text added: "STM32-C4/C8"
- board text removed: "STM32-C1"
- board text removed: "STM32-C2"
- board text removed: "STM32-C3"
- board text removed: "STM32-C4"

Commit message: em producao
Parts:
- added L+3.3v1: LED Yelow, LED_THT:LED_D5.0mm, F.Cu at (113.3, 140.0)
- added R1: 510, Resistor_THT:R_Axial_DIN0207_L6.3mm_D2.5mm_P7.62mm_Horizontal, F.Cu at (113.3, 126.5)
Routing:
- net Earth: track 388.8 -> 331.9 mm
- net 3.3V_step: track 111.6 -> 134.8 mm, vias 1 -> 2
- net Net-(L+3.3v1-A): track 0.00 -> 3.30 mm
