File: KiCadProjects/Aquisicao/Aquisicao_STM_barramento_V01/Aquisicao_STM_Barramento_v01.kicad_sch (KiCad schematic)
At the start: 13 parts, among them J1 alimentacao analogica, J2 sinais analogicos, J3 comunicacao / sinais digitais, J4 Conn_01x02, U1 BluePill_STM32F103C, U2 LM2596S-5, U3 LM1117T-3.3

Commit message: modificar
Parts:
- added J5: Conn_01x02, symbol Connector_Generic:Conn_01x02
- added U4, U5, U6: BluePill_STM32F103C, BluePill_breakouts:BluePill_STM32F103C, symbol bluepill_breakouts:BluePill_STM32F103C
Connections:
- net 3.3V_step: now also U4.40 (VCC3V3), U5.40 (VCC3V3), U6.40 (VCC3V3)
- net Ampl1: now also U1.6 (PA1), U4.6 (PA1), U5.6 (PA1), U6.6 (PA1); no longer U1.13 (PB0)
- net Ampl2: now also U1.9 (PA4), U4.9 (PA4), U5.9 (PA4), U6.9 (PA4); no longer U1.14 (PB1)
- net Earth: now also U4.20 (GND), U5.20 (GND), U6.20 (GND)
- net SCL1: now also U4.36 (PB8), U5.36 (PB8), U6.36 (PB8)
- net SDA1: now also U4.37 (PB9), U5.37 (PB9), U6.37 (PB9)
- net SINCD: now also U1.3 (PC14), U4.3 (PC14), U5.3 (PC14), U6.3 (PC14)
- net SINC_A: now also U1.10 (PA5_SCK1), U4.10 (PA5_SCK1), U5.10 (PA5_SCK1), U6.10 (PA5_SCK1)
- net SINC_B: now also U1.11 (PA6_MISO1), U4.11 (PA6_MISO1), U5.11 (PA6_MISO1), U6.11 (PA6_MISO1)
- net SINC_C: now also U1.12 (PA7_MOSI1), U4.12 (PA7_MOSI1), U5.12 (PA7_MOSI1), U6.12 (PA7_MOSI1)
- net sign_E1: now also U4.5 (PA0)
- new net sign_E2: J5.1 (Pin_1), U5.5 (PA0)
- new net sign_E3: J5.2 (Pin_2), U6.5 (PA0)
Other:
- moved on the sheet: J4, U1

Commit message: tmp
Parts:
- added U5A1: 74HC4051, 74HC4051N:N16, symbol 74xx:74HC4051
- added U7: BluePill_STM32F103C, BluePill_breakouts:BluePill_STM32F103C, symbol bluepill_breakouts:BluePill_STM32F103C
Connections:
- net D6: now reaches J3.10 (Pin_10)
- net D6: now also U5A1.5 (A5)
- net D5: now reaches J3.11 (Pin_11)
- net D5: now also U5A1.1 (A4)
- net D4: now reaches J3.12 (Pin_12)
- net D4: now also U5A1.12 (A3)
- net D3: now reaches J3.13 (Pin_13)
- net D3: now also U5A1.15 (A2)
- net D2: now reaches J3.14 (Pin_14)
- net D2: now also U5A1.14 (A1)
- net D1: now reaches J3.15 (Pin_15)
- net D1: now also U5A1.13 (A0)
- net D8: now reaches J3.8 (Pin_8)
- net D8: now also U5A1.4 (A7)
- net D7: now reaches J3.9 (Pin_9)
- net D7: now also U5A1.2 (A6)
- new net S0: U5A1.11 (S0)
- new net S1: U5A1.10 (S1)
- new net S2: U5A1.9 (S2)
- new net Ẽ: U5A1.6 (~{E})
Other:
- note added: "STM controlador geral"
- note added: "Sinais digitais controle eletrodos"
- moved on the sheet: J3, U1

Commit message: tmp
Parts:
- removed U5A1: 74HC4051, 74HC4051N:N16, symbol 74xx:74HC4051
- removed U7: BluePill_STM32F103C, BluePill_breakouts:BluePill_STM32F103C, symbol bluepill_breakouts:BluePill_STM32F103C
Connections:
- net D1 is gone; now on net SINC_A: J3.15 (Pin_15)
- net D2 is gone; now on net SINC_B: J3.14 (Pin_14)
- net D3 is gone; now on net SINC_C: J3.13 (Pin_13)
- net SCL1: now also U1.34 (PB6_SCL1), U4.34 (PB6_SCL1), U5.34 (PB6_SCL1), U6.34 (PB6_SCL1); no longer U1.36 (PB8), U4.36 (PB8), U5.36 (PB8), U6.36 (PB8)
- net SDA1: now also U1.35 (PB7_SDA1), U4.35 (PB7_SDA1), U5.35 (PB7_SDA1), U6.35 (PB7_SDA1); no longer U1.37 (PB9), U4.37 (PB9), U5.37 (PB9), U6.37 (PB9)
- net D4: no longer names the net of J3.12 (Pin_12)
- net D5: no longer names the net of J3.11 (Pin_11)
- net D6: no longer names the net of J3.10 (Pin_10)
- net D7: no longer names the net of J3.9 (Pin_9)
- net D8: no longer names the net of J3.8 (Pin_8)
Other:
- note removed: "STM controlador geral"
- note removed: "Sinais digitais controle eletrodos"
- moved on the sheet: C1, C2, C3, C4, D1, J4, J5, L1, U1, U2, U3, U4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

Commit message: tmp
Parts:
- removed J4, J5: Conn_01x02, symbol Connector_Generic:Conn_01x02
- added J4: Conn_01x04, Connector_PinHeader_2.54mm:PinHeader_1x04_P2.54mm_Horizontal, symbol Connector_Generic:Conn_01x04
- U1, U4, U5, U6: footprint BluePill_breakouts:BluePill_STM32F103C -> BluePill_STM32:BluePill_STM32F103C
Connections:
- net sign_E0 renamed sign_C1
- net sign_C1: now also J4.4 (Pin_4)
- net sign_E1 renamed sign_C2
- net sign_C2: now also J4.3 (Pin_3)
- net sign_E2 renamed sign_C3
- net sign_C3: now also J4.2 (Pin_2)
- net sign_E3 renamed sign_C4
- net sign_C4: now also J4.1 (Pin_1)
Changed lines of the file:
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@@
     )
   )
-  (global_label "sign_E3" (shape input) (at 70.358 138.43 90) (fields_autoplaced)
-    (effects (font (size 1.27 1.27)) (justify left))
-    (property "Intersheetrefs" "${INTERSHEET_REFS}" (at 70.358 128.1878 90)
+  (global_label "sign_C4" (shape input) (at 107.95 132.08 90) (fields_autoplaced)
+    (effects (font (size 1.27 1.27)) (justify left))
+    (property "Intersheetrefs" "${INTERSHEET_REFS}" (at 107.95 121.7168 90)
       (effects (font (size 1.27 1.27)) (justify left) hide)
     )
@@
     )
   )
-  (global_label "sign_E0" (shape input) (at 40.132 137.668 90) (fields_autoplaced)
-    (effects (font (size 1.27 1.27)) (justify left))
-    (property "Intersheetrefs" "${INTERSHEET_REFS}" (at 40.132 127.4258 90)
+  (global_label "sign_C1" (shape input) (at 100.33 132.08 90) (fields_autoplaced)
+    (effects (font (size 1.27 1.27)) (justify left))
+    (property "Intersheetrefs" "${INTERSHEET_REFS}" (at 100.33 121.7168 90)
       (effects (font (size 1.27 1.27)) (justify left) hide)
     )
@@
     )
   )
-  (global_label "sign_E2" (shape input) (at 67.818 138.43 90) (fields_autoplaced)
-    (effects (font (size 1.27 1.27)) (justify left))
-    (property "Intersheetrefs" "${INTERSHEET_REFS}" (at 67.818 128.1878 90)
+  (global_label "sign_C3" (shape input) (at 105.41 132.08 90) (fields_autoplaced)
+    (effects (font (size 1.27 1.27)) (justify left))
+    (property "Intersheetrefs" "${INTERSHEET_REFS}" (at 105.41 121.7168 90)
       (effects (font (size 1.27 1.27)) (justify left) hide)
     )
@@
     )
   )
-  (global_label "sign_E1" (shape input) (at 42.672 137.668 90) (fields_autoplaced)
-    (effects (font (size 1.27 1.27)) (justify left))
-    (property "Intersheetrefs" "${INTERSHEET_REFS}" (at 42.672 127.4258 90)
+  (global_label "sign_C2" (shape input) (at 102.87 132.08 90) (fields_autoplaced)
+    (effects (font (size 1.27 1.27)) (justify left))
+    (property "Intersheetrefs" "${INTERSHEET_REFS}" (at 102.87 121.7168 90)
       (effects (font (size 1.27 1.27)) (justify left) hide)
     )
@@
     )
   )
-  (global_label "sign_E1" (shape input) (at 91.694 54.864 180) (fields_autoplaced)
-    (effects (font (size 1.27 1.27)) (justify right))
-    (property "Intersheetrefs" "${INTERSHEET_REFS}" (at 81.4518 54.864 0)
+  (global_label "sign_C2" (shape input) (at 91.694 54.864 180) (fields_autoplaced)
+    (effects (font (size 1.27 1.27)) (justify right))
+    (property "Intersheetrefs" "${INTERSHEET_REFS}" (at 81.3308 54.864 0)
       (effects (font (size 1.27 1.27)) (justify right) hide)
     )
@@
     )
   )
-  (global_label "sign_E0" (shape input) (at 23.622 54.864 180) (fields_autoplaced)
-    (effects (font (size 1.27 1.27)) (justify right))
-    (property "Intersheetrefs" "${INTERSHEET_REFS}" (at 13.3798 54.864 0)
+  (global_label "sign_C1" (shape input) (at 23.622 54.864 180) (fields_autoplaced)
+    (effects (font (size 1.27 1.27)) (justify right))
+    (property "Intersheetrefs" "${INTERSHEET_REFS}" (at 13.2588 54.864 0)
       (effects (font (size 1.27 1.27)) (justify right) hide)
     )
@@
     )
   )
-  (global_label "sign_E3" (shape input) (at 225.298 55.372 180) (fields_autoplaced)
-    (effects (font (size 1.27 1.27)) (justify right))
-    (property "Intersheetrefs" "${INTERSHEET_REFS}" (at 215.0558 55.372 0)
+  (global_label "sign_C4" (shape input) (at 225.298 55.372 180) (fields_autoplaced)
+    (effects (font (size 1.27 1.27)) (justify right))
+    (property "Intersheetrefs" "${INTERSHEET_REFS}" (at 214.9348 55.372 0)
       (effects (font (size 1.27 1.27)) (justify right) hide)
     )
@@
     )
   )
-  (global_label "sign_E2" (shape input) (at 156.464 56.134 180) (fields_autoplaced)
-    (effects (font (size 1.27 1.27)) (justify right))
-    (property "Intersheetrefs" "${INTERSHEET_REFS}" (at 146.2218 56.134 0)
+  (global_label "sign_C3" (shape input) (at 156.464 56.134 180) (fields_autoplaced)
+    (effects (font (size 1.27 1.27)) (justify right))
+    (property "Intersheetrefs" "${INTERSHEET_REFS}" (at 146.1008 56.134 0)
       (effects (font (size 1.27 1.27)) (justify right) hide)
     )
@@
     )
   )
-  (symbol (lib_id "Connector_Generic:Conn_01x02") (at 40.132 142.748 90) (mirror x) (unit 1)
-    (in_bom yes) (on_board yes) (dnp no)
-    (property "Reference" "J4" (at 26.289 140.081 90)
-      (effects (font (size 1.27 1.27)) (justify right))
-    )
-    (property "Value" "Conn_01x02" (at 26.289 142.621 90)
-      (effects (font (size 1.27 1.27)) (justify right))
-    )
-    (property "Footprint" "" (at 40.132 142.748 0)
-      (effects (font (size 1.27 1.27)) hide)
-    )
-    (property "Datasheet" "~" (at 40.132 142.748 0)
-      (effects (font (size 1.27 1.27)) hide)
-    )
-    (pin "1")
-    (pin "2")
-    (instances
-      (project "Aquisicao_STM_Barramento_v01"
-        (path "/f0ff92cf-26e5-4ab9-977d-5f9689e8a5d0"
-          (reference "J4") (unit 1)
-        )
-      )
-    )
-  )
-  (symbol (lib_id "Connector_Generic:Conn_01x02") (at 67.818 143.51 90) (mirror x) (unit 1)
-    (in_bom yes) (on_board yes) (dnp no)
-    (property "Reference" "J5" (at 53.975 140.843 90)
-      (effects (font (size 1.27 1.27)) (justify right))
-    )
-    (property "Value" "Conn_01x02" (at 53.975 143.383 90)
-      (effects (font (size 1.27 1.27)) (justify right))
-    )
-    (property "Footprint" "" (at 67.818 143.51 0)
-      (effects (font (size 1.27 1.27)) hide)
-    )
-    (property "Datasheet" "~" (at 67.818 143.51 0)
-      (effects (font (size 1.27 1.27)) hide)
-    )
-    (pin "1")
-    (pin "2")
-    (instances
-      (project "Aquisicao_STM_Barramento_v01"
-        (path "/f0ff92cf-26e5-4ab9-977d-5f9689e8a5d0"
-          (reference "J5") (unit 1)
-        )
-      )
-    )
-  )
   (symbol (lib_id "bluepill_breakouts:BluePill_STM32F103C") (at 178.054 63.754 0) (unit 1)
     (in_bom yes) (on_board yes) (dnp no) (fields_autoplaced)
@@
       (effects (font (size 1.27 1.27)))
     )
-    (property "Footprint" "BluePill_breakouts:BluePill_STM32F103C" (at 179.324 104.394 0)
+    (property "Footprint" "BluePill_STM32:BluePill_STM32F103C" (at 179.324 104.394 0)
       (effects (font (size 1.27 1.27)) hide)
     )
@@
       (effects (font (size 1.27 1.27)))
     )
-    (property "Footprint" "BluePill_breakouts:BluePill_STM32F103C" (at 248.158 103.632 0)
+    (property "Footprint" "BluePill_STM32:BluePill_STM32F103C" (at 248.158 103.632 0)
       (effects (font (size 1.27 1.27)) hide)
     )
@@
       (effects (font (size 1.27 1.27)))
     )
-    (property "Footprint" "BluePill_breakouts:BluePill_STM32F103C" (at 114.554 103.124 0)
+    (property "Footprint" "BluePill_STM32:BluePill_STM32F103C" (at 114.554 103.124 0)
       (effects (font (size 1.27 1.27)) hide)
     )
@@
       (effects (font (size 1.27 1.27)))
     )
-    (property "Footprint" "BluePill_breakouts:BluePill_STM32F103C" (at 46.482 103.124 0)
+    (property "Footprint" "BluePill_STM32:BluePill_STM32F103C" (at 46.482 103.124 0)
       (effects (font (size 1.27 1.27)) hide)
     )
@@
         )
       )
+    )
+  )
+  (symbol (lib_id "Connector_Generic:Conn_01x04") (at 105.41 137.16 270) (unit 1)
+    (in_bom yes) (on_board yes) (dnp no)
+    (property "Reference" "J4" (at 104.14 140.97 90)
+      (effects (font (size 1.27 1.27)))
+    )
+    (property "Value" "Conn_01x04" (at 104.14 143.51 90)
+      (effects (font (size 1.27 1.27)))
+    )
+    (property "Footprint" "Connector_PinHeader_2.54mm:PinHeader_1x04_P2.54mm_Horizontal" (at 105.41 137.16 0)
+      (effects (font (size 1.27 1.27)) hide)
+    )
+    (property "Datasheet" "~" (at 105.41 137.16 0)
+      (effects (font (size 1.27 1.27)) hide)
+    )
+    (pin "3")
+    (pin "4")
+    (pin "1")
+    (pin "2")
+    (instances
+      (project "Aquisicao_STM_Barramento_v01"
+        (path "/f0ff92cf-26e5-4ab9-977d-5f9689e8a5d0"
+          (reference "J4") (unit 1)
+        )
+      )

Commit message: para producao
Parts:
- added J5: Conn_01x04, Connector_PinHeader_2.54mm:PinHeader_1x04_P2.54mm_Horizontal, symbol Connector_Generic:Conn_01x04
Connections:
- net SINCD: now also U1.14 (PB1), U4.14 (PB1), U5.14 (PB1), U6.14 (PB1); no longer U1.3 (PC14), U4.3 (PC14), U5.3 (PC14), U6.3 (PC14)
- net sign_C7: now reaches U5.13 (PB0)
- net sign_C7: now also J5.2 (Pin_2)
- net sign_C8: now reaches U6.13 (PB0)
- net sign_C8: now also J5.1 (Pin_1)
- net sign_C6: now reaches U4.13 (PB0)
- net sign_C6: now also J5.3 (Pin_3)
- net sign_C5: now reaches U1.13 (PB0)
- net sign_C5: now also J5.4 (Pin_4)
Other:
- moved on the sheet: U1, U4, U5, U6

Commit message: tmp
Other:
- company: EITduino -> (none)
- title: Barramento V04 -> Placa de aquisicao STM32Bluepill
Changed lines of the file:
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@@
   (paper "A4")
   (title_block
-    (title "Barramento V04")
-    (date "2024-02-05")
-    (rev "v04")
-    (company "EITduino")
+    (title "Placa de aquisicao STM32Bluepill")
+    (date "2024-07-25")
+    (rev "V01")
     (comment 1 "Autor: Gustavo Pinheiro")
-    (comment 2 "Barramento proposto para uma placa 90x100 mm")
-    (comment 3 "Placa face dupla")
-    (comment 4 "Pinos AGND e DGND")
-    (comment 5 "capacitor 100nF ceramico")
-    (comment 6 "capacitores uF tantalo")
+    (comment 2 "Baseado no barramento V04")
+    (comment 3 "Atenção: os sinais sinc_A , sinc_B e sinc_C foram adicionados ao barramento principal")
+    (comment 4 "4 Canais + amplitude de corrente ou 8 canais")
   )
   (junction (at 69.5948 172.339) (diameter 0) (color 0 0 0 0)

Commit message: em producao
Parts:
- added L+3.3v1: LED Yelow, LED_THT:LED_D5.0mm, symbol Device:LED
- added R1: 510, Resistor_THT:R_Axial_DIN0207_L6.3mm_D2.5mm_P7.62mm_Horizontal, symbol Device:R
Connections:
- net 3.3V_step: now also R1.1
- net Earth: now also L+3.3v1.1 (K)
- new net: L+3.3v1.2 (A), R1.2
Changed lines of the file:
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@@
+    (stroke (width 0) (type default))
+  )
+  (wire (pts (xy 45.466 132.588) (xy 40.894 132.588))
     (stroke (width 0) (type default))
   )
@@
     (effects (font (size 1.27 1.27)) (justify right))
     (property "Intersheetrefs" "${INTERSHEET_REFS}" (at 83.2538 73.66 0)
+      (effects (font (size 1.27 1.27)) (justify right) hide)
+    )
+  )
+  (global_label "3.3V_step" (shape input) (at 40.894 132.588 180) (fields_autoplaced)
+    (effects (font (size 1.27 1.27)) (justify right))
+    (property "Intersheetrefs" "${INTERSHEET_REFS}" (at 28.8374 132.588 0)
       (effects (font (size 1.27 1.27)) (justify right) hide)
     )
@@
         (path "/f0ff92cf-26e5-4ab9-977d-5f9689e8a5d0"
           (reference "#PWR015") (unit 1)
+        )
+      )
+    )
+  )
+  (symbol (lib_id "power:GND") (at 45.466 147.828 0) (unit 1)
+    (in_bom yes) (on_board yes) (dnp no) (fields_autoplaced)
+    (property "Reference" "#PWR036" (at 45.466 154.178 0)
+      (effects (font (size 1.27 1.27)) hide)
+    )
+    (property "Value" "GND" (at 45.466 152.146 0)
+      (effects (font (size 1.27 1.27)))
+    )
+    (property "Footprint" "" (at 45.466 147.828 0)
+      (effects (font (size 1.27 1.27)) hide)
+    )
+    (property "Datasheet" "" (at 45.466 147.828 0)
+      (effects (font (size 1.27 1.27)) hide)
+    )
+    (pin "1")
+    (instances
+      (project "Aquisicao_STM_Barramento_v01"
+        (path "/f0ff92cf-26e5-4ab9-977d-5f9689e8a5d0"
+          (reference "#PWR036") (unit 1)
         )
       )
@@
     )
   )
+  (symbol (lib_id "Device:R") (at 45.466 136.398 0) (unit 1)
+    (in_bom yes) (on_board yes) (dnp no) (fields_autoplaced)
+    (property "Reference" "R1" (at 48.133 135.128 0)
+      (effects (font (size 1.27 1.27)) (justify left))
+    )
+    (property "Value" "510" (at 48.133 137.668 0)
+      (effects (font (size 1.27 1.27)) (justify left))
+    )
+    (property "Footprint" "Resistor_THT:R_Axial_DIN0207_L6.3mm_D2.5mm_P7.62mm_Horizontal" (at 43.688 136.398 90)
+      (effects (font (size 1.27 1.27)) hide)
+    )
+    (property "Datasheet" "~" (at 45.466 136.398 0)
+      (effects (font (size 1.27 1.27)) hide)
+    )
+    (pin "2")
+    (pin "1")
+    (instances
+      (project "Aquisicao_STM_Barramento_v01"
+        (path "/f0ff92cf-26e5-4ab9-977d-5f9689e8a5d0"
+          (reference "R1") (unit 1)
+        )
+      )
+    )
+  )
   (symbol (lib_id "power:GND") (at 98.298 178.816 180) (unit 1)
     (in_bom yes) (on_board yes) (dnp no) (fields_autoplaced)
@@
         )
       )
+    )
+  )
+  (symbol (lib_id "Device:LED") (at 45.466 144.018 90) (unit 1)
+    (in_bom yes) (on_board yes) (dnp no) (fields_autoplaced)
+    (property "Reference" "L+3.3v1" (at 49.403 144.3355 90)
+      (effects (font (size 1.27 1.27)) (justify right))
+    )
+    (property "Value" "LED Yelow" (at 49.403 146.8755 90)
+      (effects (font (size 1.27 1.27)) (justify right))
+    )
+    (property "Footprint" "LED_THT:LED_D5.0mm" (at 45.466 144.018 0)
+      (effects (font (size 1.27 1.27)) hide)
+    )
+    (property "Datasheet" "~" (at 45.466 144.018 0)
+      (effects (font (size 1.27 1.27)) hide)
+    )
+    (pin "2")
+    (pin "1")
+    (instances
+      (project "Aquisicao_STM_Barramento_v01"
+        (path "/f0ff92cf-26e5-4ab9-977d-5f9689e8a5d0"
+          (reference "L+3.3v1") (unit 1)
+        )
+      )
