File: KiCadProjects/Demux/tmp/Demux_V02.kicad_pcb (KiCad board)
At the start: 2 copper layers, 90 x 100 mm, 34 parts, among them J1 alimentacao analogica, J10 +3.3Vmux, J11 -9Vmux, J12 -5Vmux, J13 GNDmux, J14 conectorEletrodos, J15 conectorEletrodos, J2 sinais analogicos, J3 comunicacao / sinais digitais, J4 Conn_01x03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

Commit message: em producao
Changed lines of the file:
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@@
     (property "ki_keywords" "R res resistor")
     (attr through_hole)
-    (fp_text reference "R4" (at 3.81 -2.37) (layer "F.SilkS")
+    (fp_text reference "R4" (at -1.952 -0.58 90) (layer "F.SilkS")
         (effects (font (size 1 1) (thickness 0.15)))
     )
@@
     (property "ki_keywords" "LED diode")
     (attr through_hole)
-    (fp_text reference "L+9v1" (at 1.27 -3.96) (layer "F.SilkS")
+    (fp_text reference "L+9v1" (at -1.714 4.246 90) (layer "F.SilkS")
         (effects (font (size 1 1) (thickness 0.15)))
     )
@@
     (property "ki_keywords" "R res resistor")
     (attr through_hole)
-    (fp_text reference "R3" (at 3.81 -2.37) (layer "F.SilkS")
+    (fp_text reference "R3" (at -1.952 -0.274 90) (layer "F.SilkS")
         (effects (font (size 1 1) (thickness 0.15)))
     )
@@
     (property "ki_keywords" "R res resistor")
     (attr through_hole)
-    (fp_text reference "R1" (at 3.81 -2.37) (layer "F.SilkS")
+    (fp_text reference "R1" (at 0.114 -2.538) (layer "F.SilkS")
         (effects (font (size 1 1) (thickness 0.15)))
     )
@@
     (effects (font (size 1 0.6) (thickness 0.15) bold) (justify left))
   )
-  (gr_text "Demux\nV01\n2024" (at 180.5 100.5 90) (layer "F.SilkS")
+  (gr_text "Demux\nV01\n2024" (at 180.5 105.156 90) (layer "F.SilkS")
     (effects (font (size 2 2) (thickness 0.3)) (justify bottom))
   )
