File: KiCadProjects/Aquisicao/Aquisicao_STM_barramento_V02/Aquisicao_STM_Barramento_v02.kicad_pcb (KiCad board)
At the start: 2 copper layers, 90 x 100 mm, 25 parts, among them J1 alimentacao analogica, J10 gpio-U1, J11 gpio-U2, J12 gpio-U3, J13 gpio-U4, J2 sinais analogicos, J3 comunicacao / sinais digitais, J4 Conn_02x08_Top_Bottom, J5 Conn_02x08_Top_Bottom, J6 Conn_02x08_Top_Bottom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

Commit message: agc
Parts:
- moved D1 3.08 mm to (112.7, 136.0)
- moved J5 2.83 mm to (153.4, 144.2)
- moved J4 2.50 mm to (131.1, 144.2)
Routing:
- net Earth: track 0.00 -> 389.2 mm, vias 0 -> 30
- net SINCD: track 0.00 -> 259.5 mm, vias 0 -> 3
- net sign_C1: track 0.00 -> 247.3 mm, vias 0 -> 4
- net Pot7_X9c10x_U/D: track 0.00 -> 236.6 mm, vias 0 -> 1
- net Pot6_X9c10x_INC: track 0.00 -> 230.6 mm, vias 0 -> 1
- net Pot8_X9c10x_U/D: track 0.00 -> 210.7 mm, vias 0 -> 2
- net sign_C4: track 0.00 -> 209.6 mm, vias 0 -> 1
- net Pot8_CS_(X9c104): track 0.00 -> 197.6 mm, vias 0 -> 1
- net Pot6_X9c10x_U/D: track 0.00 -> 190.3 mm, vias 0 -> 5
- net Pot4_X9c10x_INC: track 0.00 -> 189.3 mm, vias 0 -> 5
- net sign_C7: track 0.00 -> 168.7 mm, vias 0 -> 3
- net VCC: track 0.00 -> 167.5 mm, vias 0 -> 1
- net Pot1_X9c10x_INC: track 0.00 -> 166.6 mm, vias 0 -> 4
- net Pot4_CS_(X9c104): track 0.00 -> 164.3 mm, vias 0 -> 1
- net Pot7_X9c10x_INC: track 0.00 -> 163.8 mm, vias 0 -> 3
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- added copper zone on B.Cu, net Earth
- added copper zone on F.Cu, net Earth
