File: KiCadProjects/Aquisicao/Aquisicao_STM_barramento_V02/Aquisicao_STM_Barramento_v02.kicad_sch (KiCad schematic)
At the start: 25 parts, among them J1 alimentacao analogica, J10 gpio-U1, J11 gpio-U2, J12 gpio-U3, J13 gpio-U4, J2 sinais analogicos, J3 comunicacao / sinais digitais, J4 Conn_02x08_Top_Bottom, J5 Conn_02x08_Top_Bottom, J6 Conn_02x08_Top_Bottom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

Commit message: versao digpot
Other:
- moved on the sheet: C1, C2, C3, C4, D1, J1, J10, J11, J12, J13, J2, J3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
