File: KiCadProjects/Aquisicao/Aquisicao_STM_barramento_V03/Aquisicao_STM_Barramento_v03.kicad_pcb (KiCad board)
At the start: 2 copper layers, 90 x 100 mm, 25 parts, among them J1 alimentacao analogica, J10 gpio-U1, J11 gpio-U2, J12 gpio-U3, J13 gpio-U4, J2 sinais analogicos, J3 comunicacao / sinais digitais, J4 Conn_02x08_Top_Bottom, J5 Conn_02x08_Top_Bottom, J6 Conn_02x08_Top_Bottom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

Commit message: versao chave digital
Parts:
- removed J4, J5, J6, J7: Conn_02x08_Top_Bottom, Connector_PinHeader_2.54mm:PinHeader_2x08_P2.54mm_Horizontal
- added J14: Conn_02x05_Top_Bottom, Connector_PinHeader_2.54mm:PinHeader_2x05_P2.54mm_Horizontal, F.Cu at (124.1, 57.4)
- added J15: Conn_02x05_Top_Bottom, Connector_PinHeader_2.54mm:PinHeader_2x05_P2.54mm_Horizontal, F.Cu at (137.9, 57.5)
- added J16: Conn_02x05_Top_Bottom, Connector_PinHeader_2.54mm:PinHeader_2x05_P2.54mm_Horizontal, F.Cu at (151.8, 57.4)
- added J17: Conn_02x05_Top_Bottom, Connector_PinHeader_2.54mm:PinHeader_2x05_P2.54mm_Horizontal, F.Cu at (134.3, 144.2)
- added J18: Conn_02x05_Top_Bottom, Connector_PinHeader_2.54mm:PinHeader_2x05_P2.54mm_Horizontal, F.Cu at (148.1, 144.2)
- added J19: Conn_02x05_Top_Bottom, Connector_PinHeader_2.54mm:PinHeader_2x05_P2.54mm_Horizontal, F.Cu at (161.9, 144.2)
- added J8: Conn_02x05_Top_Bottom, Connector_PinHeader_2.54mm:PinHeader_2x05_P2.54mm_Horizontal, F.Cu at (110.4, 57.4)
- added J9: Conn_02x05_Top_Bottom, Connector_PinHeader_2.54mm:PinHeader_2x05_P2.54mm_Horizontal, F.Cu at (120.5, 144.2)
- moved C1 26.6 mm to (175.8, 124.8), turned to 90 degrees
- moved C2 21.0 mm to (179.9, 130.3), turned to 90 degrees
- moved C4 2.47 mm to (167.5, 55.7)
- moved U6 1.36 mm to (171.5, 54.0)
- moved C3 1.27 mm to (180.7, 53.4)
Connections:
- U1 pad 21: PB12-U1 -> C8_1
- U1 pad 25: PA8-U1 -> C7_1
- U1 pad 30: Pot5_X9c10x_INC -> C4_1
- U1 pad 31: Pot5_X9c10x_U/D -> C3_1
- U1 pad 32: Pot5_CS_(X9c104) -> C2_1
- U1 pad 33: Pot1_X9c10x_INC -> C1_1
- U1 pad 36: Pot1_X9c10x_U/D -> C6_1
- U1 pad 37: Pot1_CS_(X9c104) -> C5_1
- U2 pad 21: PB12-U2 -> C8_2
- U2 pad 25: PA8-U2 -> C7_2
- U2 pad 30: Pot6_X9c10x_INC -> C4_2
- U2 pad 31: Pot6_X9c10x_U/D -> C3_2
- U2 pad 32: Pot6_CS_(X9c104) -> C2_2
- U2 pad 33: Pot2_X9c10x_INC -> C1_2
- U2 pad 36: Pot2_X9c10x_U/D -> C6_2
- U2 pad 37: Pot2_CS_(X9c104) -> C5_2
- U3 pad 21: PB12-U3 -> C8_3
- U3 pad 25: PA8-U3 -> C7_3
- U3 pad 27: PA10-U3 -> unconnected-(U3-PA10_RX1-Pad27)
- U3 pad 28: PA11-U3 -> unconnected-(U3-PA11_USB_D--Pad28)
- U3 pad 29: PA12-U3 -> unconnected-(U3-PA12_USBD+-Pad29)
- U3 pad 30: Pot7_X9c10x_INC -> C4_3
- U3 pad 31: Pot7_X9c10x_U/D -> C3_3
- U3 pad 32: Pot7_CS_(X9c104) -> C2_3
- U3 pad 33: Pot3_X9c10x_INC -> C1_3
- U3 pad 36: Pot3_X9c10x_U/D -> C6_3
- U3 pad 37: Pot3_CS_(X9c104) -> C5_3
- U4 pad 21: PB12-U4 -> C8_4
- U4 pad 25: PA8-U4 -> C7_4
- U4 pad 30: Pot8_X9c10x_INC -> C4_4
- U4 pad 31: Pot8_X9c10x_U/D -> C3_4
- U4 pad 32: Pot8_CS_(X9c104) -> C2_4
- U4 pad 33: Pot4_X9c10x_INC -> C1_4
- U4 pad 36: Pot4_X9c10x_U/D -> C6_4
- U4 pad 37: Pot4_CS_(X9c104) -> C5_4
Routing:
- net Pot7_X9c10x_U/D: track 236.6 -> 0.00 mm, vias 1 -> 0
- net Pot6_X9c10x_INC: track 230.6 -> 0.00 mm, vias 1 -> 0
- net Pot8_X9c10x_U/D: track 210.7 -> 0.00 mm, vias 2 -> 0
- net C3_1: track 0.00 -> 204.2 mm, vias 0 -> 3
- net Pot8_CS_(X9c104): track 197.6 -> 0.00 mm, vias 1 -> 0
- net Pot6_X9c10x_U/D: track 190.3 -> 0.00 mm, vias 5 -> 0
- net Pot4_X9c10x_INC: track 189.3 -> 0.00 mm, vias 5 -> 0
- net C4_1: track 0.00 -> 185.5 mm, vias 0 -> 1
- net C1_1: track 0.00 -> 182.9 mm, vias 0 -> 4
- net C6_3: track 0.00 -> 175.1 mm, vias 0 -> 7
- net C8_3: track 0.00 -> 171.2 mm, vias 0 -> 5
- net C2_1: track 0.00 -> 170.2 mm, vias 0 -> 2
- net C5_3: track 0.00 -> 168.0 mm, vias 0 -> 5
- net Pot1_X9c10x_INC: track 166.6 -> 0.00 mm, vias 4 -> 0
- net Pot4_CS_(X9c104): track 164.3 -> 0.00 mm, vias 1 -> 0
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Other:
- board text added: "Aquisicao V03 2025"
- board text added: "C1_1"
- board text added: "C1_1 to C4_1"
- board text added: "C1_2"
- board text added: "C1_3"
- board text added: "C1_4"
- board text added: "C1_4 to C4_4"
- board text added: "C2_1"
- board text added: "C2_2"
- board text added: "C2_3"
- board text added: "C2_4"
- board text added: "C3_1"
- board text added: "C3_2"
- board text added: "C3_3"
- board text added: "C3_4"
- board text added: "C4_1"
- board text added: "C4_2"
- board text added: "C4_3"
- board text added: "C4_4"
- board text added: "C5_1"
- board text added: "C5_1 to C8_1"
- board text added: "C5_2"
- board text added: "C5_2 to C8_2"
- board text added: "C5_3"
- board text added: "C5_3 to C8_3"
- board text added: "C5_4"
- board text added: "C5_4 to C8_4"
- board text added: "C6_1"
- board text added: "C6_2"
- board text added: "C6_3"
- board text added: "C6_4"
- board text added: "C7_1"
- board text added: "C7_2"
- board text added: "C7_3"
- board text added: "C7_4"
- board text added: "C8_1"
- board text added: "C8_2"
- board text added: "C8_3"
- board text added: "C8_4"
- board text added: "Ch1"
- board text added: "Ch2"
- board text added: "Ch3"
- board text added: "Ch4"
- board text added: "Ch5"
- board text added: "Ch6"
- board text added: "Ch7"
- board text added: "Ch8"
- board text added: "STM32-Ch1/Ch5"
- board text added: "STM32-Ch2/Ch6"
- board text added: "STM32-Ch3/Ch7"
- board text added: "STM32-Ch4/Ch8"
- board text removed: "Aquisicao V02 2024"
- board text removed: "C1"
- board text removed: "C2"
- board text removed: "C3"
- board text removed: "C4"
- board text removed: "C5"
- board text removed: "C6"
- board text removed: "C7"
- board text removed: "C8"
- board text removed: "CS pot1"
- board text removed: "CS pot2"
- board text removed: "CS pot5"
- board text removed: "CS pot6"
- board text removed: "INC pot1"
- board text removed: "INC pot2"
- board text removed: "INC pot5"
- board text removed: "INC pot6"
- board text removed: "STM32-C1/C5"
- board text removed: "STM32-C2/C6"
- board text removed: "STM32-C3/C7"
- board text removed: "STM32-C4/C8"
- board text removed: "U/D pot1"
- board text removed: "U/D pot2"
- board text removed: "U/D pot5"
- board text removed: "U/D pot6"
- board text removed: "pot3"
- board text removed: "pot4"
- board text removed: "pot7"
- board text removed: "pot8"
