File: KiCadProjects/Aquisicao/Aquisicao_STM_barramento_V03/Aquisicao_STM_Barramento_v03.kicad_sch (KiCad schematic)
At the start: 38 parts, among them J1 alimentacao analogica, J10 gpio-U1, J11 gpio-U2, J12 gpio-U3, J13 gpio-U4, J14 In_1 select, J15 In_2 select, J16 Conn_01x04, J2 sinais analogicos, J3 comunicacao / sinais digitais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

Commit message: versao chave digital
Parts:
- removed J14, J8: In_1 select, Connector_PinHeader_2.54mm:PinHeader_1x03_P2.54mm_Vertical, symbol Connector_Generic:Conn_01x03
- removed J15, J9: In_2 select, Connector_PinHeader_2.54mm:PinHeader_1x03_P2.54mm_Vertical, symbol Connector_Generic:Conn_01x03
- removed J16: Conn_01x04, Connector_PinHeader_2.54mm:PinHeader_1x04_P2.54mm_Horizontal, symbol Connector_Generic:Conn_01x04
- removed J4, J5, J6, J7: Conn_02x08_Top_Bottom, Connector_PinHeader_2.54mm:PinHeader_2x08_P2.54mm_Horizontal, symbol Connector_Generic:Conn_02x08_Top_Bottom
- removed R2, R3: 51k, Resistor_THT:R_Axial_DIN0207_L6.3mm_D2.5mm_P7.62mm_Horizontal, symbol Device:R
- removed U1-buffer1, U2-gain1: AD828AN, AD828:N_8_ADI, symbol AD828AN:AD828AN
- removed U4-DigPot3, U5-DigPot1: X9c10x, X9c10X_module:X9c10X_module, symbol X9c10X_module:X9c10X_module
- removed U5-buffer1, U6-gain1: AD8056ARZ, AD8056ARZ:R_8_ADI, symbol AD8056ARZ:AD8056ARZ
- added J14, J15, J16, J17, J18, J19, J8, J9: Conn_02x05_Top_Bottom, Connector_PinHeader_2.54mm:PinHeader_2x05_P2.54mm_Horizontal, symbol Connector_Generic:Conn_02x05_Top_Bottom
Connections:
- net PA10-U3: no longer U3.27 (PA10_RX1)
- net PA11-U3: no longer U3.28 (PA11_USB_D-)
- net PA12-U3: no longer U3.29 (PA12_USBD+)
- net PA8-U1: no longer U1.25 (PA8)
- net PA8-U2: no longer U2.25 (PA8)
- net PA8-U3: no longer U3.25 (PA8)
- net PA8-U4: no longer U4.25 (PA8)
- net PB12-U1: no longer U1.21 (PB12)
- net PB12-U2: no longer U2.21 (PB12)
- net PB12-U3: no longer U3.21 (PB12)
- net PB12-U4: no longer U4.21 (PB12)
- net sign_C1: now also J8.10 (Pin_10), J9.10 (Pin_10)
- net sign_C2: now also J14.10 (Pin_10), J17.10 (Pin_10)
- net sign_C3: now also J15.10 (Pin_10), J18.10 (Pin_10); no longer U1.13 (PB0)
- net sign_C4: now also J16.10 (Pin_10), J19.10 (Pin_10); no longer U2.13 (PB0)
- net sign_C5: now also U1.13 (PB0), J8.9 (Pin_9), J9.9 (Pin_9)
- net sign_C6: now also U2.13 (PB0), J14.9 (Pin_9), J17.9 (Pin_9)
- net sign_C7: now also J15.9 (Pin_9), J18.9 (Pin_9)
- net sign_C8: now also J16.9 (Pin_9), J19.9 (Pin_9)
- net Pot1_CS_(X9c104) renamed C5_1
- net C5_1: now also J8.1 (Pin_1), J9.1 (Pin_1)
- net Pot1_X9c10x_INC renamed C1_1
- net C1_1: now also J8.2 (Pin_2), J9.2 (Pin_2)
- net Pot1_X9c10x_U/D renamed C6_1
- net C6_1: now also J8.3 (Pin_3), J9.3 (Pin_3)
- net Pot2_CS_(X9c104) renamed C5_2
- net C5_2: now also J14.1 (Pin_1), J17.1 (Pin_1)
- net Pot2_X9c10x_INC renamed C1_2
- net C1_2: now also J14.2 (Pin_2), J17.2 (Pin_2)
- net Pot2_X9c10x_U/D renamed C6_2
- net C6_2: now also J14.3 (Pin_3), J17.3 (Pin_3)
- net Pot3_CS_(X9c104) renamed C2_1
- net C2_1: now also J8.4 (Pin_4), J9.4 (Pin_4); no longer U3.37 (PB9)
- net Pot3_X9c10x_INC renamed C1_3
- net C1_3: now also J15.2 (Pin_2), J18.2 (Pin_2); no longer U1.30 (PA15)
- net Pot3_X9c10x_U/D renamed C3_1
- net C3_1: now also J8.6 (Pin_6), J9.6 (Pin_6); no longer U3.36 (PB8)
- net Pot4_CS_(X9c104) renamed C5_4
- net C5_4: now also J16.1 (Pin_1), J19.1 (Pin_1)
- net Pot4_X9c10x_INC renamed C1_4
- net C1_4: now also J16.2 (Pin_2), J19.2 (Pin_2)
- net Pot4_X9c10x_U/D renamed C6_4
- net C6_4: now also J16.3 (Pin_3), J19.3 (Pin_3)
- net Pot6_CS_(X9c104) renamed C2_2
- net C2_2: now also J14.4 (Pin_4), J17.4 (Pin_4)
- net Pot6_X9c10x_INC renamed C4_2
- net C4_2: now also J14.8 (Pin_8), J17.8 (Pin_8)
- net Pot6_X9c10x_U/D renamed C3_2
- net C3_2: now also J14.6 (Pin_6), J17.6 (Pin_6)
- net Pot7_CS_(X9c104) renamed C2_3
- net C2_3: now also J15.4 (Pin_4), J18.4 (Pin_4)
- net Pot7_X9c10x_INC renamed C4_3
- net C4_3: now also J15.8 (Pin_8), J18.8 (Pin_8)
- net Pot7_X9c10x_U/D renamed C3_3
- net C3_3: now also J15.6 (Pin_6), J18.6 (Pin_6)
- net Pot8_CS_(X9c104) renamed C2_4
- net C2_4: now also J16.4 (Pin_4), J19.4 (Pin_4)
- net Pot8_X9c10x_INC renamed C4_4
- net C4_4: now also J16.8 (Pin_8), J19.8 (Pin_8)
- net Pot8_X9c10x_U/D renamed C3_4
- net C3_4: now also J16.6 (Pin_6), J19.6 (Pin_6)
- new net C4_1: J8.8 (Pin_8), J9.8 (Pin_8), U1.30 (PA15)
- new net C5_3: J15.1 (Pin_1), J18.1 (Pin_1), U3.37 (PB9)
- new net C6_3: J15.3 (Pin_3), J18.3 (Pin_3), U3.36 (PB8)
- new net C7_1: J8.5 (Pin_5), J9.5 (Pin_5), U1.25 (PA8)
- new net C7_2: J14.5 (Pin_5), J17.5 (Pin_5), U2.25 (PA8)
- new net C7_3: J15.5 (Pin_5), J18.5 (Pin_5), U3.25 (PA8)
- new net C7_4: J16.5 (Pin_5), J19.5 (Pin_5), U4.25 (PA8)
- new net C8_1: J8.7 (Pin_7), J9.7 (Pin_7), U1.21 (PB12)
- new net C8_2: J14.7 (Pin_7), J17.7 (Pin_7), U2.21 (PB12)
- new net C8_3: J15.7 (Pin_7), J18.7 (Pin_7), U3.21 (PB12)
- new net C8_4: J16.7 (Pin_7), J19.7 (Pin_7), U4.21 (PB12)
Other:
- note removed: "DigPot1"
- note removed: "DigPot3"
- note removed: "G = -Rf/Rs"
- note removed: "buffer entrada"
- note removed: "ganho_programavel"
- moved on the sheet: C1, C2, C3, C4, D1, J1, J10, J11, J12, J13, J2, J3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
