File: KiCadProjects/Gerador_sinais/AD9850/V01a/Signal_generator_AD9850_V01a.kicad_sch (KiCad schematic)
At the start: 11 parts, among them J1 alimentacao analogica, J2 sinais analogicos, J3 comunicacao / sinais digitais, J4 3.3V STM32, J5 5.0V STM32, U1-AD9850 AD9850_module, U2 BluePill_STM32F103C

Commit message: versao simples sem ganho
Parts:
- removed J5: 5.0V STM32, Connector_PinHeader_2.54mm:PinHeader_1x02_P2.54mm_Vertical, symbol Connector_Generic:Conn_01x02
Connections:
- net Sin1_PA is gone; now on net Sin1: C3.2, R11.1
- net Sin2_PA is gone; now on net Sin2: C4.2, R12.1
Changed lines of the file:
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@@
 	(wire
 		(pts
-			(xy 137.033 42.037) (xy 137.033 40.894)
-		)
-		(stroke
-			(width 0)
-			(type default)
-		)
-	)
-	(wire
-		(pts
 			(xy 30.226 176.53) (xy 30.226 183.134)
 		)
@@
 	(wire
 		(pts
-			(xy 130.429 54.61) (xy 131.953 54.61)
-		)
-		(stroke
-			(width 0)
-			(type default)
-		)
-	)
-	(wire
-		(pts
 			(xy 130.429 62.23) (xy 158.242 62.23)
 		)
@@
 	(wire
 		(pts
-			(xy 131.953 54.61) (xy 131.953 42.037)
-		)
-		(stroke
-			(width 0)
-			(type default)
-		)
-	)
-	(wire
-		(pts
 			(xy 116.8388 180.34) (xy 116.8388 182.88)
 		)
@@
 	(wire
 		(pts
-			(xy 131.953 42.037) (xy 134.493 42.037)
-		)
-		(stroke
-			(width 0)
-			(type default)
-		)
-	)
-	(wire
-		(pts
 			(xy 129.54 181.773) (xy 129.54 182.88)
 		)
@@
 		)
 	)
-	(global_label "Sin2_PA"
+	(global_label "Sin2"
 		(shape input)
 		(at 211.201 73.66 0)
@@
 		)
 		(property "Intersheetrefs" "${INTERSHEET_REFS}"
-			(at 221.6852 73.66 0)
+			(at 218.359 73.66 0)
 			(effects
 				(font
@@
 		)
 	)
-	(global_label "Sin1_PA"
+	(global_label "Sin1"
 		(shape input)
 		(at 197.231 73.787 0)
@@
 		)
 		(property "Intersheetrefs" "${INTERSHEET_REFS}"
-			(at 207.7152 73.787 0)
+			(at 204.389 73.787 0)
 			(effects
 				(font
@@
 	)
 	(symbol
-		(lib_id "power:+5V")
-		(at 137.033 40.894 0)
-		(unit 1)
-		(exclude_from_sim no)
-		(in_bom yes)
-		(on_board yes)
-		(dnp no)
-		(property "Reference" "#PWR042"
-			(at 137.033 44.704 0)
-			(effects
-				(font
-					(size 1.27 1.27)
-				)
-				(hide yes)
-			)
-		)
-		(property "Value" "+5V"
-			(at 136.9789 38.3455 90)
-			(effects
-				(font
-					(size 1.27 1.27)
-				)
-				(justify left)
-			)
-		)
-		(property "Footprint" ""
-			(at 137.033 40.894 0)
-			(effects
-				(font
-					(size 1.27 1.27)
-				)
-				(hide yes)
-			)
-		)
-		(property "Datasheet" ""
-			(at 137.033 40.894 0)
-			(effects
-				(font
-					(size 1.27 1.27)
-				)
-				(hide yes)
-			)
-		)
-		(property "Description" ""
-			(at 137.033 40.894 0)
-			(effects
-				(font
-					(size 1.27 1.27)
-				)
-			)
-		)
-		(pin "1"
-		)
-		(instances
-			(project "Gerador_Sinais_AD9850"
-				(path "/f0ff92cf-26e5-4ab9-977d-5f9689e8a5d0"
-					(reference "#PWR042")
-					(unit 1)
-				)
-			)
-		)
-	)
-	(symbol
 		(lib_id "power:Earth")
 		(at 121.9171 180.9886 180)
@@
 					(unit 1)
 				)
-			)
-		)
-	)
-	(symbol
-		(lib_id "Connector_Generic:Conn_01x02")
-		(at 137.033 47.117 270)
-		(unit 1)
-		(exclude_from_sim no)
-		(in_bom yes)
-		(on_board yes)
-		(dnp no)
-		(fields_autoplaced yes)
-		(property "Reference" "J5"
-			(at 139.065 45.847 90)
-			(effects
-				(font
-					(size 1.27 1.27)
-				)
-				(justify left)
-			)
-		)
-		(property "Value" "5.0V STM32"
-			(at 139.065 48.387 90)
-			(effects
-				(font
-					(size 1.27 1.27)
-				)
-				(justify left)
-			)
-		)
-		(property "Footprint" "Connector_PinHeader_2.54mm:PinHeader_1x02_P2.54mm_Vertical"
-			(at 137.033 47.117 0)
-			(effects
-				(font
-					(size 1.27 1.27)
-				)
-				(hide yes)
-			)
-		)
-		(property "Datasheet" "~"
-			(at 137.033 47.117 0)
-			(effects
-				(font
-					(size 1.27 1.27)
-				)
-				(hide yes)
-			)
-		)
-		(property "Description" ""
-			(at 137.033 47.117 0)
-			(effects
-				(font
-					(size 1.27 1.27)
-				)
-			)
-		)
-		(pin "2"
-		)
-		(pin "1"
-		)
-		(instances
-			(project "Gerador_Sinais_AD9850"
-				(path "/f0ff92cf-26e5-4ab9-977d-5f9689e8a5d0"
-					(reference "J5")
-					(unit 1)
-				)
